File: circuit1/tia.kicad_sch (KiCad schematic)
At the start: 12 parts

Commit message: test
Parts:
- U2: renamed from U?; footprint (none) -> Package_SO:SOIC-8_3.9x4.9mm_P1.27mm
- U3: renamed from U?; footprint (none) -> Package_TO_SOT_SMD:SOT-23-6
- gave numbers to parts that had none: 8
Changed lines of the file:
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@@
   (symbol (lib_id "Device:R") (at 149.86 83.82 270) (unit 1)
     (in_bom yes) (on_board yes)
-    (property "Reference" "R?" (id 0) (at 150.114 81.534 90))
+    (property "Reference" "R5" (id 0) (at 150.114 81.534 90))
     (property "Value" "3k" (id 1) (at 149.86 83.82 90))
     (property "Footprint" "" (id 2) (at 149.86 82.042 90)
@@
   (symbol (lib_id "power:GND") (at 181.61 101.6 0) (unit 1)
     (in_bom yes) (on_board yes) (fields_autoplaced)
-    (property "Reference" "#PWR?" (id 0) (at 181.61 107.95 0)
+    (property "Reference" "#PWR0104" (id 0) (at 181.61 107.95 0)
       (effects (font (size 1.27 1.27)) hide)
     )
@@
   (symbol (lib_id "Amplifier_Operational:MCP6002-xSN") (at 46.99 59.69 0) (unit 3)
     (in_bom yes) (on_board yes) (fields_autoplaced)
-    (property "Reference" "U?" (id 0) (at 45.72 58.4199 0)
+    (property "Reference" "U2" (id 0) (at 45.72 58.4199 0)
       (effects (font (size 1.27 1.27)) (justify left))
     )
@@
       (effects (font (size 1.27 1.27)) (justify left))
     )
-    (property "Footprint" "" (id 2) (at 46.99 59.69 0)
+    (property "Footprint" "Package_SO:SOIC-8_3.9x4.9mm_P1.27mm" (id 2) (at 46.99 59.69 0)
       (effects (font (size 1.27 1.27)) hide)
     )
@@
   (symbol (lib_id "Device:C") (at 115.57 96.52 90) (unit 1)
     (in_bom yes) (on_board yes)
-    (property "Reference" "C?" (id 0) (at 115.6208 92.964 90))
+    (property "Reference" "C1" (id 0) (at 115.6208 92.964 90))
     (property "Value" "10pF" (id 1) (at 115.5192 100.076 90))
     (property "Footprint" "" (id 2) (at 119.38 95.5548 0)
@@
   (symbol (lib_id "power:+3.3V") (at 181.61 81.28 0) (unit 1)
     (in_bom yes) (on_board yes) (fields_autoplaced)
-    (property "Reference" "#PWR?" (id 0) (at 181.61 85.09 0)
+    (property "Reference" "#PWR0103" (id 0) (at 181.61 85.09 0)
       (effects (font (size 1.27 1.27)) hide)
     )
@@
   (symbol (lib_id "Device:R") (at 149.86 96.52 270) (unit 1)
     (in_bom yes) (on_board yes)
-    (property "Reference" "R?" (id 0) (at 150.114 94.234 90))
+    (property "Reference" "R6" (id 0) (at 150.114 94.234 90))
     (property "Value" "3k" (id 1) (at 149.86 96.52 90))
     (property "Footprint" "" (id 2) (at 149.86 94.742 90)
@@
   (symbol (lib_id "power:GND") (at 109.22 123.19 0) (unit 1)
     (in_bom yes) (on_board yes) (fields_autoplaced)
-    (property "Reference" "#PWR?" (id 0) (at 109.22 129.54 0)
+    (property "Reference" "#PWR0107" (id 0) (at 109.22 129.54 0)
       (effects (font (size 1.27 1.27)) hide)
     )
@@
   (symbol (lib_id "Device:R") (at 96.52 69.85 180) (unit 1)
     (in_bom yes) (on_board yes)
-    (property "Reference" "R?" (id 0) (at 99.06 68.5799 0)
+    (property "Reference" "R1" (id 0) (at 99.06 68.5799 0)
       (effects (font (size 1.27 1.27)) (justify right))
     )
@@
   (symbol (lib_id "power:GND") (at 125.73 81.28 0) (unit 1)
     (in_bom yes) (on_board yes) (fields_autoplaced)
-    (property "Reference" "#PWR?" (id 0) (at 125.73 87.63 0)
+    (property "Reference" "#PWR0102" (id 0) (at 125.73 87.63 0)
       (effects (font (size 1.27 1.27)) hide)
     )
@@
   (symbol (lib_id "Amplifier_Operational:MCP6002-xSN") (at 116.84 120.65 0) (mirror x) (unit 2)
     (in_bom yes) (on_board yes) (fields_autoplaced)
-    (property "Reference" "U?" (id 0) (at 116.84 110.49 0))
+    (property "Reference" "U2" (id 0) (at 116.84 110.49 0))
     (property "Value" "MCP6002-xSN" (id 1) (at 116.84 113.03 0))
-    (property "Footprint" "" (id 2) (at 116.84 120.65 0)
+    (property "Footprint" "Package_SO:SOIC-8_3.9x4.9mm_P1.27mm" (id 2) (at 116.84 120.65 0)
       (effects (font (size 1.27 1.27)) hide)
     )
@@
   (symbol (lib_id "power:+5V") (at 44.45 52.07 0) (unit 1)
     (in_bom yes) (on_board yes) (fields_autoplaced)
-    (property "Reference" "#PWR?" (id 0) (at 44.45 55.88 0)
+    (property "Reference" "#PWR0108" (id 0) (at 44.45 55.88 0)
       (effects (font (size 1.27 1.27)) hide)
     )
@@
   (symbol (lib_id "power:GND") (at 168.91 93.98 0) (unit 1)
     (in_bom yes) (on_board yes) (fields_autoplaced)
-    (property "Reference" "#PWR?" (id 0) (at 168.91 100.33 0)
+    (property "Reference" "#PWR0105" (id 0) (at 168.91 100.33 0)
       (effects (font (size 1.27 1.27)) hide)
     )
@@
   (symbol (lib_id "Device:R") (at 115.57 106.68 90) (unit 1)
     (in_bom yes) (on_board yes)
-    (property "Reference" "R?" (id 0) (at 115.7732 104.2924 90))
+    (property "Reference" "R2" (id 0) (at 115.7732 104.2924 90))
     (property "Value" "1M" (id 1) (at 115.57 106.68 90))
     (property "Footprint" "" (id 2) (at 115.57 108.458 90)
@@
   (symbol (lib_id "Device:R") (at 125.73 77.47 180) (unit 1)
     (in_bom yes) (on_board yes) (fields_autoplaced)
-    (property "Reference" "R?" (id 0) (at 128.27 76.1999 0)
+    (property "Reference" "R4" (id 0) (at 128.27 76.1999 0)
       (effects (font (size 1.27 1.27)) (justify right))
     )
@@
   (symbol (lib_id "power:GND") (at 158.75 100.33 0) (unit 1)
     (in_bom yes) (on_board yes) (fields_autoplaced)
-    (property "Reference" "#PWR?" (id 0) (at 158.75 106.68 0)
+    (property "Reference" "#PWR0101" (id 0) (at 158.75 106.68 0)
       (effects (font (size 1.27 1.27)) hide)
     )
@@
   (symbol (lib_id "power:GND") (at 44.45 67.31 0) (unit 1)
     (in_bom yes) (on_board yes) (fields_autoplaced)
-    (property "Reference" "#PWR?" (id 0) (at 44.45 73.66 0)
+    (property "Reference" "#PWR0109" (id 0) (at 44.45 73.66 0)
       (effects (font (size 1.27 1.27)) hide)
     )
@@
   (symbol (lib_id "Analog_ADC:MCP3421A0T-ECH") (at 181.61 91.44 0) (unit 1)
     (in_bom yes) (on_board yes) (fields_autoplaced)
-    (property "Reference" "U?" (id 0) (at 183.6294 80.01 0)
+    (property "Reference" "U3" (id 0) (at 183.6294 80.01 0)
       (effects (font (size 1.27 1.27)) (justify left))
     )
@@
       (effects (font (size 1.27 1.27)) (justify left))
     )
-    (property "Footprint" "" (id 2) (at 181.61 91.44 0)
+    (property "Footprint" "Package_TO_SOT_SMD:SOT-23-6" (id 2) (at 181.61 91.44 0)
       (effects (font (size 1.27 1.27) italic) hide)
     )
@@
   (symbol (lib_id "power:GND") (at 96.52 73.66 0) (unit 1)
     (in_bom yes) (on_board yes) (fields_autoplaced)
-    (property "Reference" "#PWR?" (id 0) (at 96.52 80.01 0)
+    (property "Reference" "#PWR0106" (id 0) (at 96.52 80.01 0)
       (effects (font (size 1.27 1.27)) hide)
     )
@@
   (symbol (lib_id "Amplifier_Operational:MCP6002-xSN") (at 118.11 66.04 0) (unit 1)
     (in_bom yes) (on_board yes) (fields_autoplaced)
-    (property "Reference" "U?" (id 0) (at 118.11 55.88 0))
+    (property "Reference" "U2" (id 0) (at 118.11 55.88 0))
     (property "Value" "MCP6002-xSN" (id 1) (at 118.11 58.42 0))
-    (property "Footprint" "" (id 2) (at 118.11 66.04 0)
+    (property "Footprint" "Package_SO:SOIC-8_3.9x4.9mm_P1.27mm" (id 2) (at 118.11 66.04 0)
       (effects (font (size 1.27 1.27)) hide)
     )
@@
   (symbol (lib_id "Device:C") (at 158.75 96.52 0) (unit 1)
     (in_bom yes) (on_board yes) (fields_autoplaced)
-    (property "Reference" "C?" (id 0) (at 162.56 95.2499 0)
+    (property "Reference" "C2" (id 0) (at 162.56 95.2499 0)
       (effects (font (size 1.27 1.27)) (justify left))
     )
@@
   (symbol (lib_id "Device:R") (at 125.73 69.85 180) (unit 1)
     (in_bom yes) (on_board yes) (fields_autoplaced)
-    (property "Reference" "R?" (id 0) (at 128.27 68.5799 0)
-      (effects (font (size 1.27 1.27)) (justify right))
-    )
+    (property "Reference" "R3" (id 0) (at 128.27 68.5799 0)
+      (effects (font (size 1.27 1.27)) (justify right))
+    )

Commit message: update
Parts:
- removed C2: C, symbol Device:C
- removed R1, R3: 100k, symbol Device:R
- removed R4: 10k, symbol Device:R
- removed R5, R6: 3k, symbol Device:R
- removed U2: MCP6002-xSN, Package_SO:SOIC-8_3.9x4.9mm_P1.27mm, symbol Amplifier_Operational:MCP6002-xSN
- removed U3: MCP3421A0T-ECH, Package_TO_SOT_SMD:SOT-23-6, symbol Analog_ADC:MCP3421A0T-ECH
- added C? (x7): 10pF, symbol Device:C
- added C? (x4): C, symbol Device:C
- added R? (x4): 3k, symbol Device:R
- added R? (x7): 1M, symbol Device:R
- added U? (x5): MCP6004, symbol Amplifier_Operational:MCP6004
Connections:
- net GND: now also C?.2, C?.2, C?.2, C?.2, R?.1, R?.1, R?.1, R?.1
- net at C1.2, R2.2: now also R?.2, U?.8
- net TIA_photovoltaic: no longer names the net of C1.1, R2.1
- net TIA_photovoltaic: now also C?.2, R?.2, U?.9 (-)
- new net: C?.2, R?.2, R?.2, U?.7
- new net: C?.1, C?.2, R?.1, R?.2, U?.2 (-)
- new net: C?.1, C?.2, R?.1, R?.2, U?.6 (-)
- new net: C?.1, C?.2, R?.1, R?.2, U?.13 (-)
- new net: C?.2, R?.2, R?.2, U?.14
- new net: C?.2, R?.2, R?.2, U?.1
- new net CH0: C?.1
- new net CH1: C?.1
- new net CH2: C?.1
- new net CH3: C?.1
- new net GNDA: U?.10 (+), U?.12 (+), U?.3 (+), U?.5 (+)
- new net OUT0: C?.1, R?.1
- new net OUT1: C?.1, R?.1
- new net OUT2: C?.1, R?.1
- new net OUT3: C?.1, R?.1
Other:
- note added: "Optional cap is for AC mode Shurtcut this cap for DC mode"
- moved on the sheet: C1, R2
