File: circuit1/namp.kicad_sch (KiCad schematic)
At the start: 1 part

Commit message: test
Parts:
- added U1: NRF52840-DONGLE, Library:MODULE_NRF52840-DONGLE, symbol NRF52840:NRF52840-DONGLE
- gave numbers to parts that had none: 1
Connections:
- new net: U1.G1 (GND), U1.G2 (GND), U1.G3 (GND)
Changed lines of the file:
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@@
   (symbol (lib_id "Connector:Screw_Terminal_01x08") (at 69.85 79.3496 180) (unit 1)
     (in_bom yes) (on_board yes) (fields_autoplaced)
-    (property "Reference" "J?" (id 0) (at 69.85 62.8396 0))
+    (property "Reference" "J1" (id 0) (at 69.85 62.8396 0))
     (property "Value" "Screw_Terminal_01x08" (id 1) (at 69.85 65.3796 0))
     (property "Footprint" "" (id 2) (at 69.85 79.3496 0)
@@
     (pin "8")
   )
+  (symbol (lib_id "NRF52840:NRF52840-DONGLE") (at 175.6156 78.4352 0) (unit 1)
+    (in_bom yes) (on_board yes) (fields_autoplaced)
+    (property "Reference" "U1" (id 0) (at 175.6156 53.34 0))
+    (property "Value" "NRF52840-DONGLE" (id 1) (at 175.6156 55.88 0))
+    (property "Footprint" "Library:MODULE_NRF52840-DONGLE" (id 2) (at 175.6156 78.4352 0)
+      (effects (font (size 1.27 1.27)) (justify left bottom) hide)
+    )
+    (property "Datasheet" "" (id 3) (at 175.6156 78.4352 0)
+      (effects (font (size 1.27 1.27)) (justify left bottom) hide)
+    )
+    (property "MAXIMUM_PACKAGE_HEIGHT" "N/A" (id 4) (at 175.6156 78.4352 0)
+      (effects (font (size 1.27 1.27)) (justify left bottom) hide)
+    )
+    (property "MANUFACTURER" "Nordic semiconductor" (id 5) (at 175.6156 78.4352 0)
+      (effects (font (size 1.27 1.27)) (justify left bottom) hide)
+    )
+    (property "STANDARD" "Manufacturer Recommendations" (id 6) (at 175.6156 78.4352 0)
+      (effects (font (size 1.27 1.27)) (justify left bottom) hide)
+    )
+    (property "PARTREV" "1.1" (id 7) (at 175.6156 78.4352 0)
+      (effects (font (size 1.27 1.27)) (justify left bottom) hide)
+    )
+    (pin "0.02")
+    (pin "0.09")
+    (pin "0.10")
+    (pin "0.13")
+    (pin "0.15")
+    (pin "0.17")
+    (pin "0.20")
+    (pin "0.22")
+    (pin "0.24")
+    (pin "0.29")
+    (pin "0.31")
+    (pin "1.00")
+    (pin "1.10")
+    (pin "1.13")
+    (pin "1.15")
+    (pin "G1")
+    (pin "G2")
+    (pin "G3")
+    (pin "OUT")
+    (pin "SWDCLK")
+    (pin "SWDIO")
+    (pin "VBUS")
+  )
   (sheet (at 102.7684 66.4464) (size 16.51 13.97) (fields_autoplaced)
     (stroke (width 0.1524) (type solid) (color 0 0 0 0))
@@
   )
   (symbol_instances
-    (path "/b7ff3da9-7842-4918-8953-02d4d40d7f9b/1fcf4402-3abf-43fc-93d9-78721d05a741"
-      (reference "#PWR?") (unit 1) (value "GND") (footprint "")
+    (path "/b7ff3da9-7842-4918-8953-02d4d40d7f9b/ce052e62-9895-4eaf-b763-02bb1f2f2fc0"
+      (reference "#PWR0101") (unit 1) (value "GND") (footprint "")
+    )
+    (path "/b7ff3da9-7842-4918-8953-02d4d40d7f9b/667ac83c-d822-438c-9f5d-2710e18e7681"
+      (reference "#PWR0102") (unit 1) (value "GND") (footprint "")
     )
     (path "/b7ff3da9-7842-4918-8953-02d4d40d7f9b/395876dc-25ca-4ac6-b54f-626217f82dba"
-      (reference "#PWR?") (unit 1) (value "+3.3V") (footprint "")
+      (reference "#PWR0103") (unit 1) (value "+3.3V") (footprint "")
+    )
+    (path "/b7ff3da9-7842-4918-8953-02d4d40d7f9b/1fcf4402-3abf-43fc-93d9-78721d05a741"
+      (reference "#PWR0104") (unit 1) (value "GND") (footprint "")
+    )
+    (path "/b7ff3da9-7842-4918-8953-02d4d40d7f9b/958363c9-4e7e-47b4-88b6-002cec8a9803"
+      (reference "#PWR0105") (unit 1) (value "GND") (footprint "")
+    )
+    (path "/b7ff3da9-7842-4918-8953-02d4d40d7f9b/e50ae05c-e860-46a9-a40f-d000a52e3442"
+      (reference "#PWR0106") (unit 1) (value "GND") (footprint "")
     )
     (path "/b7ff3da9-7842-4918-8953-02d4d40d7f9b/57b89bb3-166d-4ad0-85be-235f39fd3653"
-      (reference "#PWR?") (unit 1) (value "GND") (footprint "")
-    )
-    (path "/b7ff3da9-7842-4918-8953-02d4d40d7f9b/667ac83c-d822-438c-9f5d-2710e18e7681"
-      (reference "#PWR?") (unit 1) (value "GND") (footprint "")
+      (reference "#PWR0107") (unit 1) (value "GND") (footprint "")
     )
     (path "/b7ff3da9-7842-4918-8953-02d4d40d7f9b/8bbcd69b-f543-4ad3-8448-38196bc4df61"
-      (reference "#PWR?") (unit 1) (value "+5V") (footprint "")
-    )
-    (path "/b7ff3da9-7842-4918-8953-02d4d40d7f9b/958363c9-4e7e-47b4-88b6-002cec8a9803"
-      (reference "#PWR?") (unit 1) (value "GND") (footprint "")
-    )
-    (path "/b7ff3da9-7842-4918-8953-02d4d40d7f9b/ce052e62-9895-4eaf-b763-02bb1f2f2fc0"
-      (reference "#PWR?") (unit 1) (value "GND") (footprint "")
+      (reference "#PWR0108") (unit 1) (value "+5V") (footprint "")
     )
     (path "/b7ff3da9-7842-4918-8953-02d4d40d7f9b/d0587138-7aff-4d35-85da-166e8be0a887"
-      (reference "#PWR?") (unit 1) (value "GND") (footprint "")
-    )
-    (path "/b7ff3da9-7842-4918-8953-02d4d40d7f9b/e50ae05c-e860-46a9-a40f-d000a52e3442"
-      (reference "#PWR?") (unit 1) (value "GND") (footprint "")
+      (reference "#PWR0109") (unit 1) (value "GND") (footprint "")
     )
     (path "/b7ff3da9-7842-4918-8953-02d4d40d7f9b/36f20f2b-df3d-4bc7-a369-fb3ef715bff8"
-      (reference "C?") (unit 1) (value "10pF") (footprint "")
+      (reference "C1") (unit 1) (value "10pF") (footprint "")
     )
     (path "/b7ff3da9-7842-4918-8953-02d4d40d7f9b/f711db5e-77b0-4494-90e8-aecb55e572ba"
-      (reference "C?") (unit 1) (value "C") (footprint "")
+      (reference "C2") (unit 1) (value "C") (footprint "")
     )
     (path "/7713734c-7dce-4582-a370-d1fe16981f73"
-      (reference "J?") (unit 1) (value "Screw_Terminal_01x08") (footprint "")
+      (reference "J1") (unit 1) (value "Screw_Terminal_01x08") (footprint "")
+    )
+    (path "/b7ff3da9-7842-4918-8953-02d4d40d7f9b/60d70fa9-3d1b-45a9-9c52-21967b1f8523"
+      (reference "R1") (unit 1) (value "100k") (footprint "")
+    )
+    (path "/b7ff3da9-7842-4918-8953-02d4d40d7f9b/9ad7de90-dad3-4363-82ad-815ad6c8684b"
+      (reference "R2") (unit 1) (value "1M") (footprint "")
+    )
+    (path "/b7ff3da9-7842-4918-8953-02d4d40d7f9b/ff9f04b5-4f9e-4ac9-8790-22e4ddd6091f"
+      (reference "R3") (unit 1) (value "100k") (footprint "")
+    )
+    (path "/b7ff3da9-7842-4918-8953-02d4d40d7f9b/ad19db20-1f54-4560-8431-a27fd29f7ff7"
+      (reference "R4") (unit 1) (value "10k") (footprint "")
     )
     (path "/b7ff3da9-7842-4918-8953-02d4d40d7f9b/0737e7df-534b-4ea4-9965-1826c988f4d3"
-      (reference "R?") (unit 1) (value "3k") (footprint "")
+      (reference "R5") (unit 1) (value "3k") (footprint "")
     )
     (path "/b7ff3da9-7842-4918-8953-02d4d40d7f9b/42b72fe8-9e97-479d-ac14-742fcc9ad3b5"
-      (reference "R?") (unit 1) (value "3k") (footprint "")
+      (reference "R6") (unit 1) (value "3k") (footprint "")
     )
-    (path "/b7ff3da9-7842-4918-8953-02d4d40d7f9b/60d70fa9-3d1b-45a9-9c52-21967b1f8523"
-      (reference "R?") (unit 1) (value "100k") (footprint "")
+    (path "/7ea20839-368e-42d0-8725-47fde16d6a61"
+      (reference "U1") (unit 1) (value "NRF52840-DONGLE") (footprint "Library:MODULE_NRF52840-DONGLE")
     )
-    (path "/b7ff3da9-7842-4918-8953-02d4d40d7f9b/9ad7de90-dad3-4363-82ad-815ad6c8684b"
-      (reference "R?") (unit 1) (value "1M") (footprint "")
+    (path "/b7ff3da9-7842-4918-8953-02d4d40d7f9b/e6f86a25-2822-42e7-8a59-a03d907af09b"
+      (reference "U2") (unit 1) (value "MCP6002-xSN") (footprint "Package_SO:SOIC-8_3.9x4.9mm_P1.27mm")
     )
-    (path "/b7ff3da9-7842-4918-8953-02d4d40d7f9b/ad19db20-1f54-4560-8431-a27fd29f7ff7"
-      (reference "R?") (unit 1) (value "10k") (footprint "")
+    (path "/b7ff3da9-7842-4918-8953-02d4d40d7f9b/7d07db6c-2b6a-4a46-bd49-1e71c9b00353"
+      (reference "U2") (unit 2) (value "MCP6002-xSN") (footprint "Package_SO:SOIC-8_3.9x4.9mm_P1.27mm")
     )
-    (path "/b7ff3da9-7842-4918-8953-02d4d40d7f9b/ff9f04b5-4f9e-4ac9-8790-22e4ddd6091f"
-      (reference "R?") (unit 1) (value "100k") (footprint "")
+    (path "/b7ff3da9-7842-4918-8953-02d4d40d7f9b/3391c75e-e1c8-43aa-a009-292b4836a03b"
+      (reference "U2") (unit 3) (value "MCP6002-xSN") (footprint "Package_SO:SOIC-8_3.9x4.9mm_P1.27mm")
     )
     (path "/b7ff3da9-7842-4918-8953-02d4d40d7f9b/e4893166-0e48-43d7-aa2c-4723dbb602ea"
-      (reference "U?") (unit 1) (value "MCP3421A0T-ECH") (footprint "")
-    )
-    (path "/b7ff3da9-7842-4918-8953-02d4d40d7f9b/e6f86a25-2822-42e7-8a59-a03d907af09b"
-      (reference "U?") (unit 1) (value "MCP6002-xSN") (footprint "")
-    )
-    (path "/b7ff3da9-7842-4918-8953-02d4d40d7f9b/7d07db6c-2b6a-4a46-bd49-1e71c9b00353"
-      (reference "U?") (unit 2) (value "MCP6002-xSN") (footprint "")
-    )
-    (path "/b7ff3da9-7842-4918-8953-02d4d40d7f9b/3391c75e-e1c8-43aa-a009-292b4836a03b"
-      (reference "U?") (unit 3) (value "MCP6002-xSN") (footprint "")
+      (reference "U3") (unit 1) (value "MCP3421A0T-ECH") (footprint "Package_TO_SOT_SMD:SOT-23-6")
     )
   )

Commit message: update
Parts:
- added C1, C10, C11, C12, C13, C14, C15, C16, C2, C3, C4, C5, C6, C7, C8, C9: 10pF, Capacitor_SMD:C_0402_1005Metric_Pad0.74x0.62mm_HandSolder, symbol Device:C
- added C17, C18, C19, C20, C21, C22, C23, C24: C, Capacitor_SMD:C_0402_1005Metric_Pad0.74x0.62mm_HandSolder, symbol Device:C
- added R1, R10, R11, R12, R13, R14, R15, R16, R2, R3, R4, R5, R6, R7, R8, R9: 1M, Resistor_SMD:R_0402_1005Metric_Pad0.72x0.64mm_HandSolder, symbol Device:R
- added R17, R18, R19, R20, R21, R22, R23, R24, R25, R26: 3k, Resistor_SMD:R_0402_1005Metric_Pad0.72x0.64mm_HandSolder, symbol Device:R
- added RV1, RV2: R_Potentiometer_Trim, Potentiometer_THT:Potentiometer_Bourns_3266W_Vertical, symbol Device:R_Potentiometer_Trim
- added U2, U3: MCP6004, Package_SO:SOIC-14_3.9x8.7mm_P1.27mm, symbol Amplifier_Operational:MCP6004
- added U4: LTC2428CGTR, Library:SSOP-28_G, symbol LTC2428CGTR:LTC2428CGTR
- J1: footprint (none) -> TerminalBlock_TE-Connectivity:TerminalBlock_TE_282834-8_1x08_P2.54mm_Horizontal
Connections:
- net CH8 is gone; now on net CH7: J1.8 (Pin_8)
- net CH1: now also J1.2 (Pin_2), C2.1; no longer J1.1 (Pin_1)
- net CH2: now also J1.3 (Pin_3), C3.1; no longer J1.2 (Pin_2)
- net CH3: now also J1.4 (Pin_4), C4.1; no longer J1.3 (Pin_3)
- net CH4: now also J1.5 (Pin_5), C5.1; no longer J1.4 (Pin_4)
- net CH5: now also J1.6 (Pin_6), C6.1; no longer J1.5 (Pin_5)
- net CH6: now also J1.7 (Pin_7), C7.1; no longer J1.6 (Pin_6)
- net CH7: now also C8.1; no longer J1.7 (Pin_7)
- new net: C9.2, R17.2, R9.2, U2.8
- new net: C11.1, C3.2, R11.1, R3.2, U2.2 (-)
- new net: C11.2, R11.2, R19.2, U2.1
- new net: C15.2, R15.2, R23.2, U3.1
- new net: C15.1, C7.2, R15.1, R7.2, U3.2 (-)
- new net: C16.1, C8.2, R16.1, R8.2, U3.13 (-)
- new net: C10.1, C2.2, R10.1, R2.2, U2.6 (-)
- new net: C10.2, R10.2, R18.2, U2.7
- new net: C16.2, R16.2, R24.2, U3.14
- new net: C12.1, C4.2, R12.1, R4.2, U2.13 (-)
- new net: C13.2, R13.2, R21.2, U3.8
- new net: R25.2, R26.1, U4.26 (FO)
- new net: C14.1, C6.2, R14.1, R6.2, U3.6 (-)
- new net: C14.2, R14.2, R22.2, U3.7
- new net: C1.2, C9.1, R1.2, R9.1, U2.9 (-)
- new net: C12.2, R12.2, R20.2, U2.14
- new net: U4.4 (ADCIN), U4.7 (MUXOUT)
- new net: C13.1, C5.2, R13.1, R5.2, U3.9 (-)
- new net +3V3: R25.1, RV1.1, RV2.1, U4.2 (VCC_2), U4.8 (VCC)
- new net +5VA: U2.4 (V+), U3.4 (V+)
- new net CH0: C1.1, J1.1 (Pin_1)
- new net CS: U4.20 (*CSMUX), U4.23 (*CSADC)
- new net DIN: U4.21 (DIN)
- new net FSSET: RV1.2, U4.3 (FSSET)
- new net GNDA: C17.2, C18.2, C19.2, C20.2, C22.2, C23.2, C24.2, R1.1, R2.1, R3.1, R4.1, R6.1, R7.1, R8.1, U2.10 (+), U2.11 (V-), U2.12 (+), U2.3 (+), U2.5 (+), U3.11 (V-), U3.12 (+), U3.3 (+), U3.5 (+)
- new net GNDD: R26.2, RV1.3, RV2.3, U4.1 (GND_2), U4.16 (GND_4), U4.18 (GND_5), U4.22 (GND_6), U4.27 (GND_7), U4.28 (GND), U4.6 (GND_3)
- new net OUT0: C17.1, R17.1, U4.9 (CH0)
- new net OUT1: C18.1, R18.1, U4.10 (CH1)
- new net OUT2: C19.1, R19.1, U4.11 (CH2)
- new net OUT3: C20.1, R20.1, U4.12 (CH3)
- new net OUT4: C21.1, R21.1, U4.13 (CH4)
- new net OUT5: C22.1, R22.1, U4.14 (CH5)
- new net OUT6: C23.1, R23.1, U4.15 (CH6)
- new net OUT7: C24.1, R24.1, U4.17 (CH7)
- new net SCK: U4.19 (CLK), U4.25 (SCK)
- new net SDO: U4.24 (SDO)
- new net ZSSET: RV2.2, U4.5 (ZSSET)
Other:
- removed sheet TIA
- note added: "Antialaising low pass or bandpass filter on the ADC input and some protection because run the opamps off 5V."
- note added: "Optional cap is for AC mode Shurtcut this cap for DC mode"
- moved on the sheet: J1, U1

Commit message: update
Parts:
- added C? (x6): C, Capacitor_SMD:C_0402_1005Metric_Pad0.74x0.62mm_HandSolder, symbol Device:C
- added J?: Screw_Terminal_01x06, symbol Connector:Screw_Terminal_01x06
- added R?: 0, Resistor_SMD:R_0402_1005Metric_Pad0.72x0.64mm_HandSolder, symbol Device:R
- added U?: TXS0108EPW, Package_SO:TSSOP-20_4.4x6.5mm_P0.65mm, symbol Logic_LevelTranslator:TXS0108EPW
- added U? (x2): LP2985-5.0, Package_TO_SOT_SMD:SOT-23-5, symbol Regulator_Linear:LP2985-5.0
- R25, R26: value 3k -> 0
Connections:
- net +3V3 is gone; now on net +5V: R25.1, RV1.1, RV2.1, U4.2 (VCC_2), U4.8 (VCC)
- net +5VA: now also C?.1, J?.3 (Pin_3), U?.5 (VOUT)
- net CS: now also U1.1.13, U?.17 (B3); no longer U4.20 (*CSMUX), U4.23 (*CSADC)
- net DIN: now also U1.1.00, U?.20 (B1); no longer U4.21 (DIN)
- net GNDA: now also C21.2, R5.1, U3.10 (+), C?.2, C?.2, C?.2, J?.1 (Pin_1), J?.2 (Pin_2), U?.2 (GND)
- net GNDD: now also U1.G1 (GND), U1.G2 (GND), U1.G3 (GND), C?.2, C?.2, C?.2, J?.4 (Pin_4), J?.5 (Pin_5), U?.2 (GND)
- net SCK: now also U1.1.15, U?.16 (B4); no longer U4.19 (CLK), U4.25 (SCK)
- net SDO: now also U1.1.10, U?.18 (B2); no longer U4.24 (SDO)
- net EN_SENSOR: now reaches U1.0.20
- net EN_SENSOR: now also R?.1, U?.3 (ON/~{OFF})
- net V_REGOUT0: now reaches U1.OUT
- net V_REGOUT0: now also U?.19 (VCCB)
- net +5V: now reaches U1.VBUS
- net +5V: now also C?.1, J?.6 (Pin_6), U?.2 (VCCA), U?.5 (VOUT)
- net FSSET: no longer names the net of RV1.2, U4.3 (FSSET)
- net ZSSET: no longer names the net of RV2.2, U4.5 (ZSSET)
- new net: C?.1, U?.4 (BP) (x2)
- new net CS5V: U4.20 (*CSMUX), U4.23 (*CSADC), U?.4 (A3)
- new net DIN5V: U4.21 (DIN), U?.1 (A1)
- new net SCK5V: U4.19 (CLK), U4.25 (SCK), U?.5 (A4)
- new net SDO5V: U4.24 (SDO), U?.3 (A2)
- new net VCC: C?.1, C?.1, R?.2, U?.1 (VIN), U?.1 (VIN), U?.3 (ON/~{OFF})
Other:
- note added: "Adjust voltage measurement range with trim pot"
- note added: "Connect photodiode to GNDA and CHx"
- note added: "FO (Pin 26): Digital input which controls the ADC's notch frequencies and conversion time. When the FO pin is connected to VCC (FO = VCC), the converter uses its internal oscillator and the digital filter first null is located at 50Hz. When the FO pin is connected to GND (FO = OV), the converter uses its internal oscillator and the digital filter first null is located at 60Hz. When FO is driven b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"
- note added: "In High Voltage mode, the output from REG0 can be used to supply external circuitry from the VDD pin. The VDD output voltage is configured in the register REGOUT0 for 1.8V, 2.1V, 2.4V, 2.7V, 3.0V and 3.3V."
- note added: "Optional resistor"
- note added: "Power supply for analog"
- note added: "Power supply for digital"
- note added: "This device is an 8-bit non-inverting level translator that uses two separate configurable power-supply rails. The A port tracks the VCCA pin supply voltage. The VCCA pin accepts any supply voltage between 1.4 V and 3.6 V. The B port tracks the VCCB pin supply voltage. The VCCB pin accepts any supply voltage between 1.65 V and 5.5 V. Two input supply pins allows for low Voltage bidirectional tran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"
- note added: "When the output-enable (OE) input is low, all outputs are placed in the high-impedance (Hi-Z) state. To ensure the Hi-Z state during power-up or power- down periods, tie OE to GND through a pull-down resistor. The minimum value of the resistor is determined by the current-sourcing capability of the driver."
- moved on the sheet: C1, C10, C11, C12, C13, C14, C15, C16, C17, C18, C19, C2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

Commit message: update
Parts:
- removed C? (x6): C, Capacitor_SMD:C_0402_1005Metric_Pad0.74x0.62mm_HandSolder, symbol Device:C
- removed J?: Screw_Terminal_01x06, symbol Connector:Screw_Terminal_01x06
- removed R?: 0, Resistor_SMD:R_0402_1005Metric_Pad0.72x0.64mm_HandSolder, symbol Device:R
- removed U4: LTC2428CGTR, Library:SSOP-28_G, symbol LTC2428CGTR:LTC2428CGTR
- removed U?: TXS0108EPW, Package_SO:TSSOP-20_4.4x6.5mm_P0.65mm, symbol Logic_LevelTranslator:TXS0108EPW
- removed U? (x2): LP2985-5.0, Package_TO_SOT_SMD:SOT-23-5, symbol Regulator_Linear:LP2985-5.0
- added C25, C26, C27, C28, C29, C30, C31, C32: C, Capacitor_SMD:C_0805_2012Metric_Pad1.18x1.45mm_HandSolder, symbol Device:C
- added F1: 20mA, Fuse:Fuse_0805_2012Metric, symbol Device:Fuse
- added J2, J3: Screw_Terminal_01x04, TerminalBlock_Phoenix:TerminalBlock_Phoenix_MPT-0,5-4-2.54_1x04_P2.54mm_Horizontal, symbol Connector:Screw_Terminal_01x04
- added R27, R28, R29, R30, R31, R32: 100, Resistor_SMD:R_0805_2012Metric_Pad1.20x1.40mm_HandSolder, symbol Device:R
- added R33, R34, R35, R36: 0, Resistor_SMD:R_0805_2012Metric_Pad1.20x1.40mm_HandSolder, symbol Device:R
- added U4: MCP1501-33xSN, Package_SO:SOIC-8_3.9x4.9mm_P1.27mm, symbol Reference_Voltage:MCP1501-33xSN
- added U5: MCP3564, Library:MCP3564, symbol MCP3564:MCP3564
- C1, C10, C11, C12, C13, C14, C15, C16, C17, C18, C19, C2, C20, C21, C22, C23, C24, C3, C4, C5, C6, C7, C8, C9: footprint Capacitor_SMD:C_0402_1005Metric_Pad0.74x0.62mm_HandSolder -> Capacitor_SMD:C_0805_2012Metric_Pad1.18x1.45mm_HandSolder
- J1: footprint TerminalBlock_TE-Connectivity:TerminalBlock_TE_282834-8_1x08_P2.54mm_Horizontal -> TerminalBlock_Phoenix:TerminalBlock_Phoenix_MPT-0,5-8-2.54_1x08_P2.54mm_Horizontal
- R1, R10, R11, R12, R13, R14, R15, R16, R17, R18, R19, R2, R20, R21, R22, R23, R24, R3, R4, R5, R6, R7, R8, R9: footprint Resistor_SMD:R_0402_1005Metric_Pad0.72x0.64mm_HandSolder -> Resistor_SMD:R_0805_2012Metric_Pad1.20x1.40mm_HandSolder
- R25, R26: value 0 -> 100; footprint Resistor_SMD:R_0402_1005Metric_Pad0.72x0.64mm_HandSolder -> Resistor_SMD:R_0805_2012Metric_Pad1.20x1.40mm_HandSolder
Connections:
- net +5V: now also C26.1, C28.1, J3.4 (Pin_4), U4.1 (VDD), U4.3 (~{SHDN}); no longer R25.1, RV1.1, RV2.1
- net GNDA: now also RV1.3, RV2.3, U1.G1 (GND), U1.G2 (GND), U1.G3 (GND), C25.2, C26.2, C27.2, C28.2, C29.2, C30.2, C31.2, C32.2, J2.1 (Pin_1), J2.2 (Pin_2), J2.3 (Pin_3), J3.1 (Pin_1), J3.2 (Pin_2), J3.3 (Pin_3), R34.2, R36.2, U4.2 (GND), U4.4 (GND), U4.5 (GND), U4.6 (GND), U5.19 (DGND), U5.2 (AGND)
- net OUT0: now also U5.5 (CH0)
- net OUT1: now also U5.6 (CH1)
- net OUT2: now also U5.7 (CH2)
- net OUT3: now also U5.8 (CH3)
- net OUT4: now also U5.9 (CH4)
- net OUT5: now also U5.10 (CH5)
- net OUT6: now also U5.11 (CH6)
- net OUT7: now also U5.12 (CH7)
- net V_REGOUT0: now also C32.1, U5.20 (DVDD)
- net at RV1.2: now also R33.2, R34.1, U5.3 (REFIN-)
- net at RV2.2: now also C25.1, R35.2, R36.1, U5.4 (REFIN+)
- net at R26.1: now also U1.0.24; no longer R25.2
- net at U1.0.22: now also R25.1
- net at U1.0.29: now also R27.1
- net at U1.0.31: now also R28.1
- net +5VA renamed ADC_AVDD
- net ADC_AVDD: now also RV1.1, RV2.1, C29.1, C30.1, C31.1, F1.2, J2.4 (Pin_4), R33.1, R35.1, U5.1 (AVDD)
- net CS: no longer names the net of U1.1.13
- net CS: now also R31.1
- net DIN: no longer names the net of U1.1.00
- net DIN: now also R29.1
- removed net GNDD: R26.2, RV1.3, RV2.3, U1.G1 (GND), U1.G2 (GND), U1.G3 (GND)
- net SCK: no longer names the net of U1.1.15
- net SCK: now also R32.1
- net SDO: no longer names the net of U1.1.10
- net SDO: now also R30.1
- new net: C27.1, F1.1, U4.7 (OUT), U4.8 (FB)
- new net ADC_CS: R32.2, U5.13 (*CS)
- new net ADC_INT: R28.2, U5.17 (*IRQ/MDAT)
- new net ADC_MCK: U5.18 (MCLKIN)
- new net ADC_SCK: R31.2, U5.14 (SCK)
- new net ADC_SDI: R30.2, U5.15 (SDI)
- new net ADC_SDO: R29.2, U5.16 (SDO)
Other:
- note added: "Analog Operating Voltage AVDD 2.7 ... 3.6V Digital Operating Voltage DVDD 1.8 ... AVDD + 0.1V, DVDD ≤ 3.6V"
- note added: "The MCP1501 is a buffered voltage reference capable of sinking and sourcing 20 mA of current. The voltage reference is a low-drift bandgap-based reference. The bandgap uses chopper-based amplifiers, effectively reducing the drift to zero."
- note added: "The REFIN+ pin is the noninverting differential reference input (VREF+). The REFIN- pin is the inverting differential reference input (VREF-). For single-ended reference applications, the REFIN- pin should be directly connected to AGND. The differential reference voltage pins must respect this condition at all times: 0.6V ≤ VREF ≤ AVDD. The differential reference voltage input is given by the fol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"
- note removed: "Adjust voltage measurement range with trim pot"
- note removed: "FO (Pin 26): Digital input which controls the ADC's notch frequencies and conversion time. When the FO pin is connected to VCC (FO = VCC), the converter uses its internal oscillator and the digital filter first null is located at 50Hz. When the FO pin is connected to GND (FO = OV), the converter uses its internal oscillator and the digital filter first null is located at 60Hz. When FO is driven b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"
- note removed: "Optional resistor"
- note removed: "Power supply for analog"
- note removed: "Power supply for digital"
- note removed: "This device is an 8-bit non-inverting level translator that uses two separate configurable power-supply rails. The A port tracks the VCCA pin supply voltage. The VCCA pin accepts any supply voltage between 1.4 V and 3.6 V. The B port tracks the VCCB pin supply voltage. The VCCB pin accepts any supply voltage between 1.65 V and 5.5 V. Two input supply pins allows for low Voltage bidirectional tran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"
- note removed: "When the output-enable (OE) input is low, all outputs are placed in the high-impedance (Hi-Z) state. To ensure the Hi-Z state during power-up or power- down periods, tie OE to GND through a pull-down resistor. The minimum value of the resistor is determined by the current-sourcing capability of the driver."
- moved on the sheet: J1, U2E, U3E
