File: circuit1/namp.kicad_sch (KiCad schematic)
At the start: 79 parts, among them J1 Screw_Terminal_01x08, J2 Screw_Terminal_01x04, J3 Screw_Terminal_01x04, U1 NRF52840-DONGLE, U2 MCP6004, U3 MCP6004, U4 MCP1501-33xSN, U5 MCP3564

Commit message: update
Parts:
- removed F1: 20mA, Fuse:Fuse_0805_2012Metric, symbol Device:Fuse
- added C? (x2): 1uF, Capacitor_SMD:C_0805_2012Metric_Pad1.18x1.45mm_HandSolder, symbol Device:C
- added R? (x2): 10, symbol Device:R
- added R?: 10k, Resistor_SMD:R_0805_2012Metric_Pad1.20x1.40mm_HandSolder, symbol Device:R
- added R? (x2): 10, Resistor_SMD:R_0805_2012Metric_Pad1.20x1.40mm_HandSolder, symbol Device:R
- added R?: 100, Resistor_SMD:R_0805_2012Metric_Pad1.20x1.40mm_HandSolder, symbol Device:R
- added U?: MCP1754S-5002xCB, Package_TO_SOT_SMD:SOT-23, symbol Regulator_Linear:MCP1754S-5002xCB
- C26: value C -> 2.2µF
- C27: value C -> 300pF
- C31, C32: value C -> 0.1µF
Connections:
- net +5V: now also C?.1, R?.1, R?.1, U?.2 (VO); no longer J3.4 (Pin_4)
- net ADC_INT: now also R?.2
- net V_REGOUT0: now also R?.1, R?.1, R?.2; no longer C32.1, U5.20 (DVDD)
- net at U4.7 (OUT), U4.8 (FB): now also R?.1; no longer C27.1
- removed net ADC_AVDD: C29.1, C30.1, C31.1, J2.4 (Pin_4), R33.1, R35.1, RV1.1, RV2.1, U2.4 (V+), U3.4 (V+), U5.1 (AVDD)
- net GNDA renamed GND
- net GND: now also J2.4 (Pin_4), C?.2, C?.2, U?.1 (GND)
- new net: C30.1, R?.2, U3.4 (V+)
- new net: C29.1, R?.2, U2.4 (V+)
- new net: C32.1, R?.1, U5.20 (DVDD)
- new net: C31.1, R?.2, U5.1 (AVDD)
- new net ADC_VREF: C27.1, R33.1, R35.1, R?.2, RV1.1, RV2.1
- new net PWR_MAX16V: C?.1, J3.4 (Pin_4), U?.3 (VI)
Other:
- note added: "The MCP1754/MCP1754S also incorporates a true output current foldback. If the output load presents an excessive load due to a low-impedance short-circuit condition, the output current and voltage will fold back towards 30 mA and 0V, respectively. The output voltage and current resume normal levels when the excessive load is removed. If the overload condition is a soft overload, the MCP1754/MCP175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"
- note added: "The MCP1754/MCP1754S is a family of CMOS Low- Dropout (LDO) voltage regulators that can deliver up to 150 mA of current while consuming only 56.0 µA of quiescent current (typical). The input operating range is specified from 3.6V to 16.0V, making it an ideal choice for four to six primary cell battery-powered applications, 12V mobile applications and one to three-cell Li-Ion-powered applications."
- note added: "Transimpedance amplifier, with DC mode or AC mode"
- note removed: "Connect photodiode to GNDA and CHx"
- moved on the sheet: C26, C27, C28, C29, C30, C31, C32, J1, J2, J3, R25, R26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

Commit message: update
Parts:
- removed R?: 10, Resistor_SMD:R_0805_2012Metric_Pad1.20x1.40mm_HandSolder, symbol Device:R
- added C33, C34, C37, C39: 1uF, Capacitor_SMD:C_0603_1608Metric, symbol Device:C
- added C38, C40: 10µF, Capacitor_SMD:C_0603_1608Metric, symbol Device:C
- added R40: 10, Resistor_SMD:R_0603_1608Metric, symbol Device:R
- added U6: MCP1754S-5002xCB, Package_TO_SOT_SMD:SOT-23, symbol Regulator_Linear:MCP1754S-5002xCB
- added U8: MCP1754S-3302xCB, Package_TO_SOT_SMD:SOT-23, symbol Regulator_Linear:MCP1754S-3302xCB
- C1, C10, C11, C12, C13, C14, C15, C16, C17, C18, C19, C2, C20, C21, C22, C23, C24, C25, C26, C27, C28, C29, C3, C30, C31, C32, C4, C5, C6, C7, C8, C9: footprint Capacitor_SMD:C_0805_2012Metric_Pad1.18x1.45mm_HandSolder -> Capacitor_SMD:C_0603_1608Metric
- C35, C36: renamed from C?; footprint Capacitor_SMD:C_0805_2012Metric_Pad1.18x1.45mm_HandSolder -> Capacitor_SMD:C_0603_1608Metric
- R1, R10, R11, R12, R13, R14, R15, R16, R17, R18, R19, R2, R20, R21, R22, R23, R24, R25, R26, R27, R28, R29, R3, R30, R31, R32, R33, R34, R35, R36, R4, R5, R6, R7, R8, R9: footprint Resistor_SMD:R_0805_2012Metric_Pad1.20x1.40mm_HandSolder -> Resistor_SMD:R_0603_1608Metric
- R37, R38: renamed from R?; footprint (none) -> Resistor_SMD:R_0603_1608Metric
- R39, R41, R42: renamed from R?; footprint Resistor_SMD:R_0805_2012Metric_Pad1.20x1.40mm_HandSolder -> Resistor_SMD:R_0603_1608Metric
- gave numbers to parts that had none: 1
Connections:
- net GND: now also C33.2, C34.2, C37.2, C38.2, C39.2, C40.2, U6.1 (GND), U8.1 (GND)
- net PWR_MAX16V: now also C26.1, U4.1 (VDD), U4.3 (~{SHDN}), C33.1, C37.1, U6.3 (VI), U8.3 (VI)
- net DVDD: now reaches C32.1, R42.1, U5.20 (DVDD)
- net DVDD: now also C40.1
- net REFIN-: now reaches R33.2, R34.1, RV1.2, U5.3 (REFIN-)
- net AVDD: now reaches C31.1, U5.1 (AVDD)
- net AVDD: now also C38.1, R40.1
- net REFIN+: now reaches C25.1, R35.2, R36.1, RV2.2, U5.4 (REFIN+)
- removed net +5V: C26.1, C28.1, C36.1, R37.1, R38.1, U1.VBUS, U4.1 (VDD), U4.3 (~{SHDN}), U7.2 (VO)
- new net: C28.1, C36.1, U1.VBUS, U7.2 (VO)
- new net: C34.1, R37.1, R38.1, U6.2 (VO)
- new net: C39.1, R40.2, U8.2 (VO)
Other:
- moved on the sheet: C1, C10, C11, C12, C13, C14, C15, C16, C17, C18, C19, C2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
