File: circuit1/namp.kicad_sch (KiCad schematic)
At the start: 95 parts, among them J1 Screw_Terminal_01x08, J2 Screw_Terminal_01x04, J3 Screw_Terminal_01x04, U1 NRF52840-DONGLE, U2 MCP6004, U3 MCP6004, U4 MCP1501-33xSN, U5 MCP3564, U6 MCP1754S-5002xCB, U7 MCP1754S-5002xCB, U8 MCP1754S-3302xCB

Commit message: update
Parts:
- removed C25: C, Capacitor_SMD:C_0603_1608Metric, symbol Device:C
- removed RV1, RV2: R_Potentiometer_Trim, Potentiometer_THT:Potentiometer_Bourns_3266W_Vertical, symbol Device:R_Potentiometer_Trim
- added R43, R44, R45, R46: 10k, Resistor_SMD:R_0603_1608Metric, symbol Device:R
- R1, R2, R3, R4, R5, R6, R7, R8: value 1M -> 10k
- R33, R34, R35, R36: value 0 -> 10k
Connections:
- net GND: now also R33.2, R35.2, U5.3 (REFIN-), R43.2, R44.2, R45.2, R46.2; no longer R1.1, R2.1, R3.1, R4.1, R5.1, R6.1, R7.1, R8.1, U2.10 (+), U2.12 (+), U2.3 (+), U2.5 (+), U3.10 (+), U3.12 (+), U3.3 (+), U3.5 (+)
- net NRF_VBUS: now reaches C28.1, C36.1, U1.VBUS, U7.2 (VO)
- net at C11.1, C3.2, R11.1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: no longer R3.2
- net TIA1_V: now reaches C30.1, R38.2, U3.4 (V+)
- net TIA1_V: now also R5.1, R6.1, R7.1, R8.1
- net at C15.1, C7.2, R15.1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: no longer R7.2
- net TIA_V: now reaches C34.1, R37.1, R38.1, U6.2 (VO)
- net at C16.1, C8.2, R16.1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: no longer R8.2
- net at C10.1, C2.2, R10.1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: no longer R2.2
- net TIA0_V: now reaches C29.1, R37.2, U2.4 (V+)
- net TIA0_V: now also R1.1, R2.1, R3.1, R4.1
- net at C12.1, C4.2, R12.1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: no longer R4.2
- net at C14.1, C6.2, R14.1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: no longer R6.2
- net at C1.2, C9.1, R9.1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: no longer R1.2
- net at C13.1, C5.2, R13.1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: no longer R5.2
- net ADC_VREF renamed ADC_VREF+
- net ADC_VREF+: now also U5.4 (REFIN+); no longer R33.1, R35.1
- net AVDD renamed ADC_AVDD
- net DVDD renamed ADC_DVDD
- net ADC_DVDD: now also R41.1
- net OUT0 renamed ADC_CH0
- net OUT1 renamed ADC_CH1
- net OUT2 renamed ADC_CH2
- net OUT3 renamed ADC_CH3
- net OUT4 renamed ADC_CH4
- net OUT5 renamed ADC_CH5
- net OUT6 renamed ADC_CH6
- net OUT7 renamed ADC_CH7
- removed net REFIN+: R35.2, R36.1, U5.4 (REFIN+)
- removed net REFIN-: R33.2, R34.1, U5.3 (REFIN-)
- net V_REGOUT0 renamed NRF_REG0_V
- net NRF_REG0_V: no longer R41.1
- new net: R1.2, R33.1, U2.10 (+)
- new net: R45.1, R7.2, U3.3 (+)
- new net: R2.2, R34.1, U2.5 (+)
- new net: R3.2, R35.1, U2.3 (+)
- new net: R46.1, R8.2, U3.12 (+)
- new net: R36.1, R4.2, U2.12 (+)
- new net: R43.1, R5.2, U3.10 (+)
- new net: R44.1, R6.2, U3.5 (+)
Other:
- note added: "ADC"
- note added: "MCU"
- note added: "Power"
- note added: "Terminal"
- note added: "Voltage Reference"
- moved on the sheet: C1, C10, C11, C12, C13, C14, C15, C16, C17, C18, C19, C2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

Commit message: update
Parts:
- added J4: Conn_01x08_Female, Connector_PinSocket_2.54mm:PinSocket_1x08_P2.54mm_Vertical, symbol Connector:Conn_01x08_Female
Connections:
- net ADC_CH0: now also J4.1 (Pin_1)
- net ADC_CH1: now also J4.2 (Pin_2)
- net ADC_CH2: now also J4.3 (Pin_3)
- net ADC_CH3: now also J4.4 (Pin_4)
- net ADC_CH4: now also J4.5 (Pin_5)
- net ADC_CH5: now also J4.6 (Pin_6)
- net ADC_CH6: now also J4.7 (Pin_7)
- net ADC_CH7: now also J4.8 (Pin_8)
Changed lines of the file:
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@@
     )
+  )
+  (hierarchical_label "ADC_CH6" (shape output) (at 231.14 381 180)
+    (effects (font (size 1.27 1.27)) (justify right))
   )
   (hierarchical_label "CH2" (shape output) (at 205.74 361.95 0)
@@
     (effects (font (size 1.27 1.27)) (justify left))
   )
+  (hierarchical_label "ADC_CH5" (shape output) (at 231.14 378.46 180)
+    (effects (font (size 1.27 1.27)) (justify right))
+  )
   (hierarchical_label "CH4" (shape input) (at 21.59 270.51 180)
     (effects (font (size 1.27 1.27)) (justify right))
@@
     (effects (font (size 1.27 1.27)) (justify left))
   )
+  (hierarchical_label "ADC_CH4" (shape output) (at 231.14 375.92 180)
+    (effects (font (size 1.27 1.27)) (justify right))
+  )
   (hierarchical_label "ADC_CH7" (shape output) (at 99.06 387.35 0)
     (effects (font (size 1.27 1.27)) (justify left))
@@
     (effects (font (size 1.27 1.27)) (justify right))
   )
+  (hierarchical_label "ADC_CH1" (shape output) (at 231.14 368.3 180)
+    (effects (font (size 1.27 1.27)) (justify right))
+  )
+  (hierarchical_label "ADC_CH3" (shape output) (at 231.14 373.38 180)
+    (effects (font (size 1.27 1.27)) (justify right))
+  )
   (hierarchical_label "ADC_CH6" (shape output) (at 99.06 349.25 0)
     (effects (font (size 1.27 1.27)) (justify left))
@@
     (effects (font (size 1.27 1.27)) (justify right))
   )
+  (hierarchical_label "ADC_CH0" (shape output) (at 231.14 365.76 180)
+    (effects (font (size 1.27 1.27)) (justify right))
+  )
   (hierarchical_label "CH1" (shape input) (at 21.59 147.32 180)
     (effects (font (size 1.27 1.27)) (justify right))
@@
   (hierarchical_label "CH1" (shape output) (at 205.74 364.49 0)
     (effects (font (size 1.27 1.27)) (justify left))
+  )
+  (hierarchical_label "ADC_CH2" (shape output) (at 231.14 370.84 180)
+    (effects (font (size 1.27 1.27)) (justify right))
+  )
+  (hierarchical_label "ADC_CH7" (shape output) (at 231.14 383.54 180)
+    (effects (font (size 1.27 1.27)) (justify right))
   )
   (hierarchical_label "ADC_CH1" (shape output) (at 99.06 149.86 0)
@@
     (pin "1")
     (pin "2")
+  )
+  (symbol (lib_id "Connector:Conn_01x08_Female") (at 236.22 373.38 0) (unit 1)
+    (in_bom yes) (on_board yes) (fields_autoplaced)
+    (property "Reference" "J4" (id 0) (at 237.49 373.3799 0)
+      (effects (font (size 1.27 1.27)) (justify left))
+    )
+    (property "Value" "Conn_01x08_Female" (id 1) (at 237.49 375.9199 0)
+      (effects (font (size 1.27 1.27)) (justify left))
+    )
+    (property "Footprint" "Connector_PinSocket_2.54mm:PinSocket_1x08_P2.54mm_Vertical" (id 2) (at 236.22 373.38 0)
+      (effects (font (size 1.27 1.27)) hide)
+    )
+    (property "Datasheet" "~" (id 3) (at 236.22 373.38 0)
+      (effects (font (size 1.27 1.27)) hide)
+    )
+    (pin "1")
+    (pin "2")
+    (pin "3")
+    (pin "4")
+    (pin "5")
+    (pin "6")
+    (pin "7")
+    (pin "8")
   )
   (symbol (lib_id "power:GND") (at 173.99 361.95 90) (unit 1)
@@
       (reference "J3") (unit 1) (value "Screw_Terminal_01x04") (footprint "TerminalBlock_Phoenix:TerminalBlock_Phoenix_MPT-0,5-4-2.54_1x04_P2.54mm_Horizontal")
     )
+    (path "/5688283d-42e1-47c0-90d8-46cb5b72985d"
+      (reference "J4") (unit 1) (value "Conn_01x08_Female") (footprint "Connector_PinSocket_2.54mm:PinSocket_1x08_P2.54mm_Vertical")
+    )
     (path "/0a4670fe-f411-47c9-8912-2ac7b841eb8f"

Commit message: update
Parts:
- J4: footprint Connector_PinSocket_2.54mm:PinSocket_1x08_P2.54mm_Vertical -> Connector_PinHeader_2.54mm:PinHeader_1x08_P2.54mm_Vertical
Connections:
- net ADC_CH0: now also C19.1, R19.1; no longer C17.1, R17.1
- net ADC_CH1: now also C20.1, R20.1; no longer C18.1, R18.1
- net ADC_CH2: now also C17.1, R17.1; no longer C19.1, R19.1
- net ADC_CH3: now also C18.1, R18.1; no longer C20.1, R20.1
- net ADC_CH4: now also C23.1, R23.1; no longer C21.1, R21.1
- net ADC_CH5: now also C24.1, R24.1; no longer C22.1, R22.1
- net ADC_CH6: now also C21.1, R21.1; no longer C23.1, R23.1
- net ADC_CH7: now also C22.1, R22.1; no longer C24.1, R24.1
- net CH0: now also C3.1; no longer C1.1
- net CH1: now also C4.1; no longer C2.1
- net CH2: now also C1.1; no longer C3.1
- net CH3: now also C2.1; no longer C4.1
- net CH4: now also C7.1; no longer C5.1
- net CH5: now also C8.1; no longer C6.1
- net CH6: now also C5.1; no longer C7.1
- net CH7: now also C6.1; no longer C8.1
Changed lines of the file:
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@@
     (effects (font (size 1.27 1.27)) (justify left))
   )
-  (hierarchical_label "CH7" (shape input) (at 21.59 384.81 180)
+  (hierarchical_label "CH7" (shape input) (at 21.59 308.61 180)
     (effects (font (size 1.27 1.27)) (justify right))
   )
@@
     (effects (font (size 1.27 1.27)) (justify right))
   )
-  (hierarchical_label "CH4" (shape input) (at 21.59 270.51 180)
+  (hierarchical_label "CH4" (shape input) (at 21.59 346.71 180)
     (effects (font (size 1.27 1.27)) (justify right))
   )
@@
     (effects (font (size 1.27 1.27)) (justify left))
   )
-  (hierarchical_label "CH0" (shape input) (at 21.59 109.22 180)
+  (hierarchical_label "CH0" (shape input) (at 21.59 185.42 180)
     (effects (font (size 1.27 1.27)) (justify right))
   )
@@
     (effects (font (size 1.27 1.27)) (justify right))
   )
-  (hierarchical_label "ADC_CH7" (shape output) (at 99.06 387.35 0)
+  (hierarchical_label "ADC_CH7" (shape output) (at 99.06 311.15 0)
     (effects (font (size 1.27 1.27)) (justify left))
   )
@@
     (effects (font (size 1.27 1.27)) (justify right))
   )
-  (hierarchical_label "CH6" (shape input) (at 21.59 346.71 180)
+  (hierarchical_label "CH6" (shape input) (at 21.59 270.51 180)
     (effects (font (size 1.27 1.27)) (justify right))
   )
-  (hierarchical_label "CH5" (shape input) (at 21.59 308.61 180)
+  (hierarchical_label "CH5" (shape input) (at 21.59 384.81 180)
     (effects (font (size 1.27 1.27)) (justify right))
   )
@@
     (effects (font (size 1.27 1.27)) (justify right))
   )
-  (hierarchical_label "ADC_CH6" (shape output) (at 99.06 349.25 0)
+  (hierarchical_label "ADC_CH6" (shape output) (at 99.06 273.05 0)
     (effects (font (size 1.27 1.27)) (justify left))
   )
@@
     (effects (font (size 1.27 1.27)) (justify right))
   )
-  (hierarchical_label "ADC_CH5" (shape output) (at 99.06 311.15 0)
+  (hierarchical_label "ADC_CH5" (shape output) (at 99.06 387.35 0)
     (effects (font (size 1.27 1.27)) (justify left))
   )
@@
     (effects (font (size 1.27 1.27)) (justify right))
   )
-  (hierarchical_label "CH1" (shape input) (at 21.59 147.32 180)
+  (hierarchical_label "CH1" (shape input) (at 21.59 223.52 180)
     (effects (font (size 1.27 1.27)) (justify right))
   )
@@
     (effects (font (size 1.27 1.27)) (justify right))
   )
-  (hierarchical_label "CH3" (shape input) (at 21.59 223.52 180)
+  (hierarchical_label "CH3" (shape input) (at 21.59 147.32 180)
     (effects (font (size 1.27 1.27)) (justify right))
   )
@@
     (effects (font (size 1.27 1.27)) (justify left))
   )
-  (hierarchical_label "ADC_CH0" (shape output) (at 99.06 111.76 0)
+  (hierarchical_label "ADC_CH0" (shape output) (at 99.06 187.96 0)
     (effects (font (size 1.27 1.27)) (justify left))
   )
@@
     (effects (font (size 1.27 1.27)) (justify left))
   )
-  (hierarchical_label "ADC_CH3" (shape output) (at 99.06 226.06 0)
+  (hierarchical_label "ADC_CH3" (shape output) (at 99.06 149.86 0)
     (effects (font (size 1.27 1.27)) (justify left))
   )
-  (hierarchical_label "ADC_CH4" (shape output) (at 99.06 273.05 0)
+  (hierarchical_label "ADC_CH4" (shape output) (at 99.06 349.25 0)
     (effects (font (size 1.27 1.27)) (justify left))
   )
@@
     (effects (font (size 1.27 1.27)) (justify right))
   )
-  (hierarchical_label "CH2" (shape input) (at 21.59 185.42 180)
+  (hierarchical_label "CH2" (shape input) (at 21.59 109.22 180)
     (effects (font (size 1.27 1.27)) (justify right))
   )
@@
     (effects (font (size 1.27 1.27)) (justify right))
   )
-  (hierarchical_label "ADC_CH1" (shape output) (at 99.06 149.86 0)
+  (hierarchical_label "ADC_CH1" (shape output) (at 99.06 226.06 0)
     (effects (font (size 1.27 1.27)) (justify left))
   )
-  (hierarchical_label "ADC_CH2" (shape output) (at 99.06 187.96 0)
+  (hierarchical_label "ADC_CH2" (shape output) (at 99.06 111.76 0)
     (effects (font (size 1.27 1.27)) (justify left))
   )
@@
       (effects (font (size 1.27 1.27)) (justify left))
     )
-    (property "Footprint" "Connector_PinSocket_2.54mm:PinSocket_1x08_P2.54mm_Vertical" (id 2) (at 236.22 373.38 0)
+    (property "Footprint" "Connector_PinHeader_2.54mm:PinHeader_1x08_P2.54mm_Vertical" (id 2) (at 236.22 373.38 0)
       (effects (font (size 1.27 1.27)) hide)
     )
@@
     )
     (path "/5688283d-42e1-47c0-90d8-46cb5b72985d"
-      (reference "J4") (unit 1) (value "Conn_01x08_Female") (footprint "Connector_PinSocket_2.54mm:PinSocket_1x08_P2.54mm_Vertical")
+      (reference "J4") (unit 1) (value "Conn_01x08_Female") (footprint "Connector_PinHeader_2.54mm:PinHeader_1x08_P2.54mm_Vertical")
     )
     (path "/0a4670fe-f411-47c9-8912-2ac7b841eb8f"

Commit message: update
Parts:
- added J5: Conn_01x08_Male, Connector_PinHeader_2.54mm:PinHeader_1x08_P2.54mm_Vertical, symbol Connector:Conn_01x08_Male
Connections:
- net ADC_CS: now also J5.8 (Pin_8)
- net ADC_DVDD: now also J5.2 (Pin_2)
- net ADC_INT: now also J5.4 (Pin_4)
- net ADC_MCK: now also J5.3 (Pin_3)
- net ADC_SCK: now also J5.7 (Pin_7)
- net ADC_SDI: now also J5.6 (Pin_6)
- net ADC_SDO: now also J5.5 (Pin_5)
- net GND: now also J5.1 (Pin_1)
Changed lines of the file:
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@@
+    )
+  )
+  (global_label "ADC_SCK" (shape input) (at 560.07 290.83 0) (fields_autoplaced)
+    (effects (font (size 1.27 1.27)) (justify left))
+    (property "Intersheet References" "${INTERSHEET_REFS}" (id 0) (at 570.8288 290.7506 0)
+      (effects (font (size 1.27 1.27)) (justify left) hide)
     )
   )
@@
     )
   )
+  (global_label "ADC_MCK" (shape input) (at 560.07 280.67 0) (fields_autoplaced)
+    (effects (font (size 1.27 1.27)) (justify left))
+    (property "Intersheet References" "${INTERSHEET_REFS}" (id 0) (at 571.0707 280.5906 0)
+      (effects (font (size 1.27 1.27)) (justify left) hide)
+    )
+  )
   (global_label "ADC_INT" (shape input) (at 234.95 123.19 0) (fields_autoplaced)
     (effects (font (size 1.27 1.27)) (justify left))
@@
     )
   )
+  (global_label "ADC_CS" (shape input) (at 560.07 293.37 0) (fields_autoplaced)
+    (effects (font (size 1.27 1.27)) (justify left))
+    (property "Intersheet References" "${INTERSHEET_REFS}" (id 0) (at 569.5588 293.2906 0)
+      (effects (font (size 1.27 1.27)) (justify left) hide)
+    )
+  )
+  (global_label "ADC_INT" (shape input) (at 560.07 283.21 0) (fields_autoplaced)
+    (effects (font (size 1.27 1.27)) (justify left))
+    (property "Intersheet References" "${INTERSHEET_REFS}" (id 0) (at 569.9821 283.1306 0)
+      (effects (font (size 1.27 1.27)) (justify left) hide)
+    )
+  )
+  (global_label "ADC_SDO" (shape input) (at 560.07 285.75 0) (fields_autoplaced)
+    (effects (font (size 1.27 1.27)) (justify left))
+    (property "Intersheet References" "${INTERSHEET_REFS}" (id 0) (at 570.8893 285.6706 0)
+      (effects (font (size 1.27 1.27)) (justify left) hide)
+    )
+  )
   (global_label "TIA1_V" (shape input) (at 30.48 317.5 180) (fields_autoplaced)
     (effects (font (size 1.27 1.27)) (justify right))
@@
     )
   )
+  (global_label "ADC_SDI" (shape input) (at 560.07 288.29 0) (fields_autoplaced)
+    (effects (font (size 1.27 1.27)) (justify left))
+    (property "Intersheet References" "${INTERSHEET_REFS}" (id 0) (at 570.1636 288.2106 0)
+      (effects (font (size 1.27 1.27)) (justify left) hide)
+    )
+  )
   (global_label "ADC_SDO" (shape input) (at 234.95 125.73 0) (fields_autoplaced)
     (effects (font (size 1.27 1.27)) (justify left))
@@
     (effects (font (size 1.27 1.27)) (justify left))
     (property "Intersheet References" "${INTERSHEET_REFS}" (id 0) (at 244.4388 133.2706 0)
+      (effects (font (size 1.27 1.27)) (justify left) hide)
+    )
+  )
+  (global_label "ADC_DVDD" (shape input) (at 560.07 278.13 0) (fields_autoplaced)
+    (effects (font (size 1.27 1.27)) (justify left))
+    (property "Intersheet References" "${INTERSHEET_REFS}" (id 0) (at 571.9779 278.2094 0)
       (effects (font (size 1.27 1.27)) (justify left) hide)
     )
@@
     (pin "1")
   )
+  (symbol (lib_id "Connector:Conn_01x08_Male") (at 554.99 283.21 0) (unit 1)
+    (in_bom yes) (on_board yes) (fields_autoplaced)
+    (property "Reference" "J5" (id 0) (at 555.625 270.51 0))
+    (property "Value" "Conn_01x08_Male" (id 1) (at 555.625 273.05 0))
+    (property "Footprint" "Connector_PinHeader_2.54mm:PinHeader_1x08_P2.54mm_Vertical" (id 2) (at 554.99 283.21 0)
+      (effects (font (size 1.27 1.27)) hide)
+    )
+    (property "Datasheet" "~" (id 3) (at 554.99 283.21 0)
+      (effects (font (size 1.27 1.27)) hide)
+    )
+    (pin "1")
+    (pin "2")
+    (pin "3")
+    (pin "4")
+    (pin "5")
+    (pin "6")
+    (pin "7")
+    (pin "8")
+  )
   (symbol (lib_id "Device:R") (at 77.47 187.96 270) (unit 1)
     (in_bom yes) (on_board yes)
@@
     (pin "13")
     (pin "14")
+  )
+  (symbol (lib_id "power:GNDD") (at 560.07 275.59 90) (unit 1)
+    (in_bom yes) (on_board yes)
+    (property "Reference" "#PWR0115" (id 0) (at 566.42 275.59 0)
+      (effects (font (size 1.27 1.27)) hide)
+    )
+    (property "Value" "GNDD" (id 1) (at 562.61 275.59 90)
+      (effects (font (size 1.27 1.27)) (justify right))
+    )
+    (property "Footprint" "" (id 2) (at 560.07 275.59 0)
+      (effects (font (size 1.27 1.27)) hide)
+    )
+    (property "Datasheet" "" (id 3) (at 560.07 275.59 0)
+      (effects (font (size 1.27 1.27)) hide)
+    )
+    (pin "1")
   )
   (symbol (lib_id "power:GNDD") (at 163.83 381 0) (unit 1)
@@
       (reference "#PWR0114") (unit 1) (value "GNDD") (footprint "")
     )
+    (path "/34238737-e2f4-4660-8dc4-f6374bb15abf"
+      (reference "#PWR0115") (unit 1) (value "GNDD") (footprint "")
+    )
     (path "/1f7471b5-dfd9-4156-b85a-3ecaede73fff"
       (reference "#PWR0116") (unit 1) (value "GNDA") (footprint "")
@@
       (reference "J4") (unit 1) (value "Conn_01x08_Female") (footprint "Connector_PinHeader_2.54mm:PinHeader_1x08_P2.54mm_Vertical")
     )
+    (path "/1763f786-dd71-4840-968a-c65e7d3470b9"
+      (reference "J5") (unit 1) (value "Conn_01x08_Male") (footprint "Connector_PinHeader_2.54mm:PinHeader_1x08_P2.54mm_Vertical")
+    )
     (path "/0a4670fe-f411-47c9-8912-2ac7b841eb8f"
