File: circuit1/namp.kicad_sch (KiCad schematic)
At the start: 98 parts, among them J1 Screw_Terminal_01x08, J2 Screw_Terminal_01x04, J3 Screw_Terminal_01x04, J4 Conn_01x08_Female, J5 Conn_01x08_Male, U1 NRF52840-DONGLE, U2 MCP6004, U3 MCP6004, U4 MCP1501-33xSN, U5 MCP3564, U6 MCP1754S-5002xCB, U7 MCP1754S-5002xCB, U8 MCP1754S-3302xCB

Commit message: update
Parts:
- removed R26, R27, R29: 100, Resistor_SMD:R_0603_1608Metric, symbol Device:R
Connections:
- net ADC_CS: now also R30.2; no longer R32.2
- net ADC_SDI: now also R32.2; no longer R30.2
- net ADC_SDO: now also R25.2
- net at U1.0.29: now also R25.1
- net at U1.0.22: no longer R25.1
Changed lines of the file:
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@@
     (stroke (width 0) (type default) (color 0 0 0 0))
   )
-  (wire (pts (xy 220.98 115.57) (xy 218.44 115.57))
-    (stroke (width 0) (type default) (color 0 0 0 0))
-  )
   (wire (pts (xy 29.21 45.72) (xy 29.21 44.45))
     (stroke (width 0) (type default) (color 0 0 0 0))
@@
     (stroke (width 0) (type default) (color 0 0 0 0))
   )
-  (polyline (pts (xy 177.8 76.2) (xy 292.1 76.2))
+  (polyline (pts (xy 152.4 76.2) (xy 292.1 76.2))
     (stroke (width 0) (type default) (color 0 0 0 0))
   )
@@
     (stroke (width 0) (type default) (color 0 0 0 0))
   )
+  (wire (pts (xy 228.6 120.65) (xy 234.95 120.65))
+    (stroke (width 0) (type default) (color 0 0 0 0))
+  )
   (wire (pts (xy 21.59 308.61) (xy 29.21 308.61))
     (stroke (width 0) (type default) (color 0 0 0 0))
@@
     (stroke (width 0) (type default) (color 0 0 0 0))
   )
-  (polyline (pts (xy 177.8 76.2) (xy 177.8 152.4))
+  (polyline (pts (xy 152.4 76.2) (xy 152.4 152.4))
     (stroke (width 0) (type default) (color 0 0 0 0))
   )
@@
     (stroke (width 0) (type default) (color 0 0 0 0))
   )
-  (wire (pts (xy 228.6 125.73) (xy 234.95 125.73))
-    (stroke (width 0) (type default) (color 0 0 0 0))
-  )
   (wire (pts (xy 425.45 267.97) (xy 436.88 267.97))
     (stroke (width 0) (type default) (color 0 0 0 0))
@@
     (stroke (width 0) (type default) (color 0 0 0 0))
   )
-  (polyline (pts (xy 292.1 152.4) (xy 177.8 152.4))
+  (polyline (pts (xy 292.1 152.4) (xy 152.4 152.4))
     (stroke (width 0) (type default) (color 0 0 0 0))
   )
@@
     (stroke (width 0) (type default) (color 0 0 0 0))
   )
-  (wire (pts (xy 220.98 120.65) (xy 218.44 120.65))
-    (stroke (width 0) (type default) (color 0 0 0 0))
-  )
   (wire (pts (xy 46.99 232.41) (xy 48.26 232.41))
     (stroke (width 0) (type default) (color 0 0 0 0))
@@
     (stroke (width 0) (type default) (color 0 0 0 0))
   )
-  (wire (pts (xy 220.98 118.11) (xy 218.44 118.11))
-    (stroke (width 0) (type default) (color 0 0 0 0))
-  )
   (wire (pts (xy 52.07 330.2) (xy 49.53 330.2))
     (stroke (width 0) (type default) (color 0 0 0 0))
@@
     (stroke (width 0) (type default) (color 0 0 0 0))
   )
-  (wire (pts (xy 220.98 125.73) (xy 218.44 125.73))
-    (stroke (width 0) (type default) (color 0 0 0 0))
-  )
   (wire (pts (xy 36.83 346.71) (xy 49.53 346.71))
     (stroke (width 0) (type default) (color 0 0 0 0))
@@
     (stroke (width 0) (type default) (color 0 0 0 0))
   )
+  (wire (pts (xy 220.98 120.65) (xy 218.44 120.65))
+    (stroke (width 0) (type default) (color 0 0 0 0))
+  )
   (wire (pts (xy 170.18 381) (xy 170.18 378.46))
     (stroke (width 0) (type default) (color 0 0 0 0))
@@
     )
   )
-  (global_label "ADC_SCK" (shape input) (at 560.07 290.83 0) (fields_autoplaced)
+  (global_label "ADC_SDO" (shape input) (at 234.95 120.65 0) (fields_autoplaced)
     (effects (font (size 1.27 1.27)) (justify left))
-    (property "Intersheet References" "${INTERSHEET_REFS}" (id 0) (at 570.8288 290.7506 0)
+    (property "Intersheet References" "${INTERSHEET_REFS}" (id 0) (at 245.7693 120.5706 0)
       (effects (font (size 1.27 1.27)) (justify left) hide)
     )
   )
-  (global_label "ADC_SDI" (shape input) (at 234.95 128.27 0) (fields_autoplaced)
+  (global_label "ADC_SCK" (shape input) (at 560.07 290.83 0) (fields_autoplaced)
     (effects (font (size 1.27 1.27)) (justify left))
-    (property "Intersheet References" "${INTERSHEET_REFS}" (id 0) (at 245.0436 128.1906 0)
+    (property "Intersheet References" "${INTERSHEET_REFS}" (id 0) (at 570.8288 290.7506 0)
       (effects (font (size 1.27 1.27)) (justify left) hide)
     )
@@
     )
   )
+  (global_label "ADC_CS" (shape input) (at 234.95 128.27 0) (fields_autoplaced)
+    (effects (font (size 1.27 1.27)) (justify left))
+    (property "Intersheet References" "${INTERSHEET_REFS}" (id 0) (at 244.4388 128.1906 0)
+      (effects (font (size 1.27 1.27)) (justify left) hide)
+    )
+  )
   (global_label "ADC_CS" (shape input) (at 560.07 293.37 0) (fields_autoplaced)
     (effects (font (size 1.27 1.27)) (justify left))
@@
     )
   )
+  (global_label "ADC_SDI" (shape input) (at 234.95 133.35 0) (fields_autoplaced)
+    (effects (font (size 1.27 1.27)) (justify left))
+    (property "Intersheet References" "${INTERSHEET_REFS}" (id 0) (at 245.0436 133.2706 0)
+      (effects (font (size 1.27 1.27)) (justify left) hide)
+    )
+  )
   (global_label "ADC_SDO" (shape input) (at 560.07 285.75 0) (fields_autoplaced)
     (effects (font (size 1.27 1.27)) (justify left))
@@
     )
   )
-  (global_label "ADC_SDO" (shape input) (at 234.95 125.73 0) (fields_autoplaced)
-    (effects (font (size 1.27 1.27)) (justify left))
-    (property "Intersheet References" "${INTERSHEET_REFS}" (id 0) (at 245.7693 125.6506 0)
-      (effects (font (size 1.27 1.27)) (justify left) hide)
-    )
-  )
   (global_label "NRF_REG0_V" (shape input) (at 561.34 251.46 0) (fields_autoplaced)
     (effects (font (size 1.27 1.27)) (justify left))
@@
     )
   )
-  (global_label "ADC_CS" (shape input) (at 234.95 133.35 0) (fields_autoplaced)
-    (effects (font (size 1.27 1.27)) (justify left))
-    (property "Intersheet References" "${INTERSHEET_REFS}" (id 0) (at 244.4388 133.2706 0)
-      (effects (font (size 1.27 1.27)) (justify left) hide)
-    )
-  )
   (global_label "ADC_DVDD" (shape input) (at 560.07 278.13 0) (fields_autoplaced)
     (effects (font (size 1.27 1.27)) (justify left))
@@
     (pin "1")
   )
+  (symbol (lib_id "Device:R") (at 224.79 120.65 90) (unit 1)
+    (in_bom yes) (on_board yes)
+    (property "Reference" "R25" (id 0) (at 231.14 120.65 90))
+    (property "Value" "100" (id 1) (at 224.79 120.65 90))
+    (property "Footprint" "Resistor_SMD:R_0603_1608Metric" (id 2) (at 224.79 122.428 90)
+      (effects (font (size 1.27 1.27)) hide)
+    )
+    (property "Datasheet" "~" (id 3) (at 224.79 120.65 0)
+      (effects (font (size 1.27 1.27)) hide)
+    )
+    (pin "1")
+    (pin "2")
+  )
   (symbol (lib_id "power:GNDA") (at 242.57 355.6 90) (unit 1)
     (in_bom yes) (on_board yes) (fields_autoplaced)
@@
     (pin "1")
   )
-  (symbol (lib_id "Device:R") (at 224.79 120.65 90) (unit 1)
-    (in_bom yes) (on_board yes)
-    (property "Reference" "R27" (id 0) (at 231.14 120.65 90))
-    (property "Value" "100" (id 1) (at 224.79 120.65 90))
-    (property "Footprint" "Resistor_SMD:R_0603_1608Metric" (id 2) (at 224.79 122.428 90)
-      (effects (font (size 1.27 1.27)) hide)
-    )
-    (property "Datasheet" "~" (id 3) (at 224.79 120.65 0)
-      (effects (font (size 1.27 1.27)) hide)
-    )
-    (pin "1")
-    (pin "2")
-  )
   (symbol (lib_id "Device:C") (at 33.02 147.32 90) (unit 1)
     (in_bom yes) (on_board yes)
@@
     (pin "2")
   )
-  (symbol (lib_id "Device:R") (at 224.79 118.11 90) (unit 1)
-    (in_bom yes) (on_board yes)
-    (property "Reference" "R26" (id 0) (at 231.14 118.11 90))
-    (property "Value" "100" (id 1) (at 224.79 118.11 90))
-    (property "Footprint" "Resistor_SMD:R_0603_1608Metric" (id 2) (at 224.79 119.888 90)
-      (effects (font (size 1.27 1.27)) hide)
-    )
-    (property "Datasheet" "~" (id 3) (at 224.79 118.11 0)
-      (effects (font (size 1.27 1.27)) hide)
-    )
-    (pin "1")
-    (pin "2")
-  )
   (symbol (lib_id "Connector:Conn_01x08_Female") (at 236.22 373.38 0) (unit 1)
     (in_bom yes) (on_board yes) (fields_autoplaced)
@@
     (pin "14")
   )
-  (symbol (lib_id "Device:R") (at 224.79 125.73 90) (unit 1)
-    (in_bom yes) (on_board yes)
-    (property "Reference" "R29" (id 0) (at 231.14 125.73 90))
-    (property "Value" "100" (id 1) (at 224.79 125.73 90))
-    (property "Footprint" "Resistor_SMD:R_0603_1608Metric" (id 2) (at 224.79 127.508 90)
-      (effects (font (size 1.27 1.27)) hide)
-    )
-    (property "Datasheet" "~" (id 3) (at 224.79 125.73 0)
-      (effects (font (size 1.27 1.27)) hide)
-    )
-    (pin "1")
-    (pin "2")
-  )
   (symbol (lib_id "Amplifier_Operational:MCP6004") (at 57.15 111.76 0) (mirror x) (unit 3)
     (in_bom yes) (on_board yes)
@@
     (pin "2")
   )
-  (symbol (lib_id "Device:R") (at 224.79 115.57 90) (unit 1)
-    (in_bom yes) (on_board yes)
-    (property "Reference" "R25" (id 0) (at 231.14 115.57 90))
-    (property "Value" "100" (id 1) (at 224.79 115.57 90))
-    (property "Footprint" "Resistor_SMD:R_0603_1608Metric" (id 2) (at 224.79 117.348 90)
-      (effects (font (size 1.27 1.27)) hide)
-    )
-    (property "Datasheet" "~" (id 3) (at 224.79 115.57 0)
-      (effects (font (size 1.27 1.27)) hide)
-    )
-    (pin "1")
-    (pin "2")
-  )
   (symbol (lib_id "Device:C") (at 106.68 62.23 0) (unit 1)
     (in_bom yes) (on_board yes) (fields_autoplaced)
@@
       (reference "R24") (unit 1) (value "3k") (footprint "Resistor_SMD:R_0603_1608Metric")
     )
-    (path "/f3048abe-7448-4f1b-88e5-a5ecee64c4c3"
+    (path "/07034251-a9a7-4596-941f-8a3f95aded82"
       (reference "R25") (unit 1) (value "100") (footprint "Resistor_SMD:R_0603_1608Metric")
     )
-    (path "/5508d357-b41e-4be0-b808-648f918ff269"
-      (reference "R26") (unit 1) (value "100") (footprint "Resistor_SMD:R_0603_1608Metric")
-    )
-    (path "/4a7d2d5e-2b6b-4e3f-9654-e47cbcfddf02"
-      (reference "R27") (unit 1) (value "100") (footprint "Resistor_SMD:R_0603_1608Metric")
-    )
     (path "/94353048-5474-4735-b703-76ec6ed09c1f"
       (reference "R28") (unit 1) (value "100") (footprint "Resistor_SMD:R_0603_1608Metric")
     )
-    (path "/86968ef3-9da3-4a0d-bf8d-7527e302f32f"
-      (reference "R29") (unit 1) (value "100") (footprint "Resistor_SMD:R_0603_1608Metric")
-    )
     (path "/dbbdd361-70b7-472a-b923-f659e2536132"

Commit message: update
Parts:
- added R26: 10, Resistor_SMD:R_0603_1608Metric, symbol Device:R
Connections:
- net PWR_MAX16V: no longer C26.1, U4.1 (VDD), U4.3 (~{SHDN})
- net TIA_V renamed TIA_5V
- net TIA_5V: now also R26.1
- new net: C26.1, R26.2, U4.1 (VDD), U4.3 (~{SHDN})
- no-connect marks 0 -> 12
Changed lines of the file:
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@@
   (junction (at 49.53 377.19) (diameter 0) (color 0 0 0 0)
   )
+  (no_connect (at 218.44 118.11))
+  (no_connect (at 218.44 115.57))
+  (no_connect (at 187.96 130.81))
+  (no_connect (at 187.96 128.27))
+  (no_connect (at 187.96 125.73))
+  (no_connect (at 187.96 123.19))
+  (no_connect (at 187.96 110.49))
+  (no_connect (at 187.96 107.95))
+  (no_connect (at 218.44 125.73))
+  (no_connect (at 187.96 115.57))
+  (no_connect (at 187.96 120.65))
+  (no_connect (at 187.96 118.11))
   (polyline (pts (xy 115.57 407.67) (xy 12.7 407.67))
     (stroke (width 0) (type default) (color 0 0 0 0))
@@
     (stroke (width 0) (type default) (color 0 0 0 0))
   )
-  (wire (pts (xy 318.77 261.62) (xy 323.85 261.62))
+  (wire (pts (xy 321.31 261.62) (xy 323.85 261.62))
     (stroke (width 0) (type default) (color 0 0 0 0))
   )
@@
     (stroke (width 0) (type default) (color 0 0 0 0))
   )
+  (wire (pts (xy 307.34 261.62) (xy 313.69 261.62))
+    (stroke (width 0) (type default) (color 0 0 0 0))
+  )
   (wire (pts (xy 163.83 378.46) (xy 163.83 381))
     (stroke (width 0) (type default) (color 0 0 0 0))
@@
     )
   )
-  (global_label "TIA_V" (shape input) (at 91.44 34.29 0) (fields_autoplaced)
+  (global_label "TIA_5V" (shape input) (at 91.44 34.29 0) (fields_autoplaced)
     (effects (font (size 1.27 1.27)) (justify left))
-    (property "Intersheet References" "${INTERSHEET_REFS}" (id 0) (at 98.5702 34.2106 0)
+    (property "Intersheet References" "${INTERSHEET_REFS}" (id 0) (at 99.7798 34.2106 0)
       (effects (font (size 1.27 1.27)) (justify left) hide)
     )
@@
     )
   )
-  (global_label "PWR_MAX16V" (shape input) (at 318.77 261.62 180) (fields_autoplaced)
-    (effects (font (size 1.27 1.27)) (justify right))
-    (property "Intersheet References" "${INTERSHEET_REFS}" (id 0) (at 304.1407 261.6994 0)
-      (effects (font (size 1.27 1.27)) (justify right) hide)
-    )
-  )
   (global_label "ADC_MCK" (shape input) (at 560.07 280.67 0) (fields_autoplaced)
     (effects (font (size 1.27 1.27)) (justify left))
@@
     )
   )
+  (global_label "TIA_5V" (shape input) (at 307.34 261.62 180) (fields_autoplaced)
+    (effects (font (size 1.27 1.27)) (justify right))
+    (property "Intersheet References" "${INTERSHEET_REFS}" (id 0) (at 299.0002 261.5406 0)
+      (effects (font (size 1.27 1.27)) (justify right) hide)
+    )
+  )
   (global_label "PWR_MAX16V" (shape input) (at 27.94 34.29 180) (fields_autoplaced)
     (effects (font (size 1.27 1.27)) (justify right))
@@
     (pin "2")
   )
+  (symbol (lib_id "Device:R") (at 317.5 261.62 90) (unit 1)
+    (in_bom yes) (on_board yes) (fields_autoplaced)
+    (property "Reference" "R26" (id 0) (at 317.5 255.8879 90))
+    (property "Value" "10" (id 1) (at 317.5 258.4279 90))
+    (property "Footprint" "Resistor_SMD:R_0603_1608Metric" (id 2) (at 317.5 263.398 90)
+      (effects (font (size 1.27 1.27)) hide)
+    )
+    (property "Datasheet" "~" (id 3) (at 317.5 261.62 0)
+      (effects (font (size 1.27 1.27)) hide)
+    )
+    (pin "1")
+    (pin "2")
+  )
   (symbol (lib_id "power:GNDA") (at 242.57 355.6 90) (unit 1)
     (in_bom yes) (on_board yes) (fields_autoplaced)
@@
       (reference "R25") (unit 1) (value "100") (footprint "Resistor_SMD:R_0603_1608Metric")
     )
+    (path "/0714050a-acff-463d-b343-5ee952a83e96"
+      (reference "R26") (unit 1) (value "10") (footprint "Resistor_SMD:R_0603_1608Metric")
+    )
     (path "/94353048-5474-4735-b703-76ec6ed09c1f"

Commit message: Changed to 0805
Parts:
- C1, C10, C11, C12, C13, C14, C15, C16, C17, C18, C19, C2, C20, C21, C22, C23, C24, C26, C27, C28, C29, C3, C30, C31, C32, C33, C34, C35, C36, C37, C38, C39, C4, C40, C5, C6, C7, C8, C9: footprint Capacitor_SMD:C_0603_1608Metric -> Capacitor_SMD:C_0805_2012Metric_Pad1.18x1.45mm_HandSolder
- R1, R10, R11, R12, R13, R14, R15, R16, R17, R18, R19, R2, R20, R21, R22, R23, R24, R25, R26, R28, R3, R30, R31, R32, R33, R34, R35, R36, R37, R38, R39, R4, R40, R41, R42, R43, R44, R45, R46, R5, R6, R7, R8, R9: footprint Resistor_SMD:R_0603_1608Metric -> Resistor_SMD:R_0805_2012Metric_Pad1.20x1.40mm_HandSolder

Commit message: update
Connections:
- net ADC_CH6: now also U5.12 (CH7); no longer U5.11 (CH6)
- net ADC_CH7: now also U5.11 (CH6); no longer U5.12 (CH7)
Changed lines of the file:
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@@
     (effects (font (size 1.27 1.27)) (justify left))
   )
-  (hierarchical_label "ADC_CH6" (shape output) (at 494.03 288.29 0)
+  (hierarchical_label "ADC_CH6" (shape output) (at 494.03 285.75 0)
     (effects (font (size 1.27 1.27)) (justify left))
   )
@@
     (effects (font (size 1.27 1.27)) (justify left))
   )
-  (hierarchical_label "ADC_CH7" (shape output) (at 494.03 285.75 0)
+  (hierarchical_label "ADC_CH7" (shape output) (at 494.03 288.29 0)
     (effects (font (size 1.27 1.27)) (justify left))
   )
