File: circuit1/namp.kicad_sch (KiCad schematic)
At the start: 96 parts, among them J1 Screw_Terminal_01x08, J2 Screw_Terminal_01x04, J3 Screw_Terminal_01x04, J4 Conn_01x08_Female, J5 Conn_01x08_Male, U1 NRF52840-DONGLE, U2 MCP6004, U3 MCP6004, U4 MCP1501-33xSN, U5 MCP3564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

Commit message: update
Connections:
- net ADC_CH6: now also U5.11 (CH6); no longer U5.12 (CH7)
- net ADC_CH7: now also U5.12 (CH7); no longer U5.11 (CH6)
Changed lines of the file:
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@@
     (effects (font (size 1.27 1.27)) (justify left))
   )
-  (hierarchical_label "ADC_CH6" (shape output) (at 494.03 285.75 0)
+  (hierarchical_label "ADC_CH6" (shape output) (at 494.03 288.29 0)
     (effects (font (size 1.27 1.27)) (justify left))
   )
@@
     (effects (font (size 1.27 1.27)) (justify left))
   )
-  (hierarchical_label "ADC_CH7" (shape output) (at 494.03 288.29 0)
+  (hierarchical_label "ADC_CH7" (shape output) (at 494.03 285.75 0)
     (effects (font (size 1.27 1.27)) (justify left))
   )
