File: circuit1/namp.kicad_pcb (KiCad board)
At the start: 2 copper layers, 3 parts, among them U1 NRF52840-DONGLE, U2 MCP6002-xSN, U3 MCP3421A0T-ECH

Commit message: update
Parts:
- added C1: 10pF, Capacitor_SMD:C_0402_1005Metric_Pad0.74x0.62mm_HandSolder, F.Cu at (106.7, 73.7)
- added C10: 10pF, Capacitor_SMD:C_0402_1005Metric_Pad0.74x0.62mm_HandSolder, F.Cu at (103.5, 74.0)
- added C11: 10pF, Capacitor_SMD:C_0402_1005Metric_Pad0.74x0.62mm_HandSolder, F.Cu at (103.5, 79.9)
- added C12: 10pF, Capacitor_SMD:C_0402_1005Metric_Pad0.74x0.62mm_HandSolder, F.Cu at (118.7, 63.5)
- added C13: 10pF, Capacitor_SMD:C_0402_1005Metric_Pad0.74x0.62mm_HandSolder, F.Cu at (112.2, 71.4)
- added C14: 10pF, Capacitor_SMD:C_0402_1005Metric_Pad0.74x0.62mm_HandSolder, F.Cu at (103.5, 75.9)
- added C15: 10pF, Capacitor_SMD:C_0402_1005Metric_Pad0.74x0.62mm_HandSolder, F.Cu at (112.2, 69.4)
- added C16: 10pF, Capacitor_SMD:C_0402_1005Metric_Pad0.74x0.62mm_HandSolder, F.Cu at (97.1, 74.0)
- added C17: C, Capacitor_SMD:C_0402_1005Metric_Pad0.74x0.62mm_HandSolder, F.Cu at (103.5, 77.9)
- added C18: C, Capacitor_SMD:C_0402_1005Metric_Pad0.74x0.62mm_HandSolder, F.Cu at (112.2, 67.4)
- added C19: C, Capacitor_SMD:C_0402_1005Metric_Pad0.74x0.62mm_HandSolder, F.Cu at (93.8, 79.9)
- added C2: 10pF, Capacitor_SMD:C_0402_1005Metric_Pad0.74x0.62mm_HandSolder, F.Cu at (97.0, 78.0)
- added C20: C, Capacitor_SMD:C_0402_1005Metric_Pad0.74x0.62mm_HandSolder, F.Cu at (100.3, 77.9)
- added C21: C, Capacitor_SMD:C_0402_1005Metric_Pad0.74x0.62mm_HandSolder, F.Cu at (90.6, 79.9)
- added C22: C, Capacitor_SMD:C_0402_1005Metric_Pad0.74x0.62mm_HandSolder, F.Cu at (142.7, 45.1)
- added C23: C, Capacitor_SMD:C_0402_1005Metric_Pad0.74x0.62mm_HandSolder, F.Cu at (106.7, 75.6)
- added C24: C, Capacitor_SMD:C_0402_1005Metric_Pad0.74x0.62mm_HandSolder, F.Cu at (100.3, 76.0)
- added C3: 10pF, Capacitor_SMD:C_0402_1005Metric_Pad0.74x0.62mm_HandSolder, F.Cu at (100.4, 72.0)
- added C4: 10pF, Capacitor_SMD:C_0402_1005Metric_Pad0.74x0.62mm_HandSolder, F.Cu at (115.4, 69.3)
- added C5: 10pF, Capacitor_SMD:C_0402_1005Metric_Pad0.74x0.62mm_HandSolder, F.Cu at (106.7, 77.6)
- added C6: 10pF, Capacitor_SMD:C_0402_1005Metric_Pad0.74x0.62mm_HandSolder, F.Cu at (100.3, 79.9)
- added C7: 10pF, Capacitor_SMD:C_0402_1005Metric_Pad0.74x0.62mm_HandSolder, F.Cu at (93.8, 78.0)
- added C8: 10pF, Capacitor_SMD:C_0402_1005Metric_Pad0.74x0.62mm_HandSolder, F.Cu at (90.6, 78.0)
- added C9: 10pF, Capacitor_SMD:C_0402_1005Metric_Pad0.74x0.62mm_HandSolder, F.Cu at (97.0, 79.9)
- added J1: Screw_Terminal_01x08, TerminalBlock_TE-Connectivity:TerminalBlock_TE_282834-8_1x08_P2.54mm_Horizontal, F.Cu at (156.2, 61.0)
- added R1: 1M, Resistor_SMD:R_0402_1005Metric_Pad0.72x0.64mm_HandSolder, F.Cu at (93.9, 72.0)
- added R10: 1M, Resistor_SMD:R_0402_1005Metric_Pad0.72x0.64mm_HandSolder, F.Cu at (87.4, 73.7)
- added R11: 1M, Resistor_SMD:R_0402_1005Metric_Pad0.72x0.64mm_HandSolder, F.Cu at (80.9, 76.0)
- added R12: 1M, Resistor_SMD:R_0402_1005Metric_Pad0.72x0.64mm_HandSolder, F.Cu at (84.2, 80.0)
- added R13: 1M, Resistor_SMD:R_0402_1005Metric_Pad0.72x0.64mm_HandSolder, F.Cu at (90.7, 76.0)
- added R14: 1M, Resistor_SMD:R_0402_1005Metric_Pad0.72x0.64mm_HandSolder, F.Cu at (80.9, 78.0)
- added R15: 1M, Resistor_SMD:R_0402_1005Metric_Pad0.72x0.64mm_HandSolder, F.Cu at (80.9, 74.0)
- added R16: 1M, Resistor_SMD:R_0402_1005Metric_Pad0.72x0.64mm_HandSolder, F.Cu at (80.9, 80.0)
- added R17: 3k, Resistor_SMD:R_0402_1005Metric_Pad0.72x0.64mm_HandSolder, F.Cu at (80.9, 72.0)
- added R18: 3k, Resistor_SMD:R_0402_1005Metric_Pad0.72x0.64mm_HandSolder, F.Cu at (115.4, 63.5)
- added R19: 3k, Resistor_SMD:R_0402_1005Metric_Pad0.72x0.64mm_HandSolder, F.Cu at (112.2, 63.5)
- added R2: 1M, Resistor_SMD:R_0402_1005Metric_Pad0.72x0.64mm_HandSolder, F.Cu at (84.2, 74.0)
- added R20: 3k, Resistor_SMD:R_0402_1005Metric_Pad0.72x0.64mm_HandSolder, F.Cu at (97.2, 72.0)
- added R21: 3k, Resistor_SMD:R_0402_1005Metric_Pad0.72x0.64mm_HandSolder, F.Cu at (84.2, 76.0)
- added R22: 3k, Resistor_SMD:R_0402_1005Metric_Pad0.72x0.64mm_HandSolder, F.Cu at (87.4, 77.7)
- added R23: 3k, Resistor_SMD:R_0402_1005Metric_Pad0.72x0.64mm_HandSolder, F.Cu at (84.2, 78.0)
- added R24: 3k, Resistor_SMD:R_0402_1005Metric_Pad0.72x0.64mm_HandSolder, F.Cu at (112.2, 65.5)
- added R25: 3k, Resistor_SMD:R_0402_1005Metric_Pad0.72x0.64mm_HandSolder, F.Cu at (115.4, 67.3)
- added R26: 3k, Resistor_SMD:R_0402_1005Metric_Pad0.72x0.64mm_HandSolder, F.Cu at (90.7, 74.0)
- added R3: 1M, Resistor_SMD:R_0402_1005Metric_Pad0.72x0.64mm_HandSolder, F.Cu at (93.9, 76.0)
- added R4: 1M, Resistor_SMD:R_0402_1005Metric_Pad0.72x0.64mm_HandSolder, F.Cu at (139.4, 45.2)
- added R5: 1M, Resistor_SMD:R_0402_1005Metric_Pad0.72x0.64mm_HandSolder, F.Cu at (93.9, 74.0)
- added R6: 1M, Resistor_SMD:R_0402_1005Metric_Pad0.72x0.64mm_HandSolder, F.Cu at (84.2, 72.0)
- added R7: 1M, Resistor_SMD:R_0402_1005Metric_Pad0.72x0.64mm_HandSolder, F.Cu at (90.7, 72.0)
- added R8: 1M, Resistor_SMD:R_0402_1005Metric_Pad0.72x0.64mm_HandSolder, F.Cu at (87.4, 75.7)
- added R9: 1M, Resistor_SMD:R_0402_1005Metric_Pad0.72x0.64mm_HandSolder, F.Cu at (87.4, 79.6)
- added RV1: R_Potentiometer_Trim, Potentiometer_THT:Potentiometer_Bourns_3266W_Vertical, F.Cu at (63.5, 109.2)
- added RV2: R_Potentiometer_Trim, Potentiometer_THT:Potentiometer_Bourns_3266W_Vertical, F.Cu at (86.4, 111.8)
- added U4: LTC2428CGTR, Library:SSOP-28_G, F.Cu at (97.2, 55.9)
- U2: value MCP6002-xSN -> MCP6004; footprint Package_SO:SOIC-8_3.9x4.9mm_P1.27mm -> Package_SO:SOIC-14_3.9x8.7mm_P1.27mm
- U3: value MCP3421A0T-ECH -> MCP6004; footprint Package_TO_SOT_SMD:SOT-23-6 -> Package_SO:SOIC-14_3.9x8.7mm_P1.27mm
- moved U1 102.4 mm to (81.3, 35.6)
- moved U3 18.0 mm to (157.4, 86.4)
- moved U2 18.0 mm to (157.5, 101.6)
Connections:
- U2 pad 3: /TIA/TIA_photoconductive -> GNDA
- U2 pad 4: GND -> +5VA
- U2 pad 5: GND -> GNDA
- U2 pad 6: /TIA/TIA_photovoltaic -> Net-(C10-Pad1)
- U2 pad 8: +5V -> Net-(C9-Pad2)
- U3 pad 2: GND -> Net-(C15-Pad1)
- U3 pad 3: /TIA/SCL -> GNDA
- U3 pad 4: /TIA/SDA -> +5VA
- U3 pad 5: +3V3 -> GNDA
- U3 pad 6: GND -> Net-(C14-Pad1)

Commit message: update
Parts:
- added C25: C, Capacitor_SMD:C_0805_2012Metric_Pad1.18x1.45mm_HandSolder, F.Cu at (141.6, 99.8)
- added C26: C, Capacitor_SMD:C_0805_2012Metric_Pad1.18x1.45mm_HandSolder, F.Cu at (172.7, 96.5)
- added C27: C, Capacitor_SMD:C_0805_2012Metric_Pad1.18x1.45mm_HandSolder, F.Cu at (177.5, 93.5)
- added C28: C, Capacitor_SMD:C_0805_2012Metric_Pad1.18x1.45mm_HandSolder, F.Cu at (182.3, 93.5)
- added C29: C, Capacitor_SMD:C_0805_2012Metric_Pad1.18x1.45mm_HandSolder, F.Cu at (172.7, 99.5)
- added C30: C, Capacitor_SMD:C_0805_2012Metric_Pad1.18x1.45mm_HandSolder, F.Cu at (177.5, 99.5)
- added C31: C, Capacitor_SMD:C_0805_2012Metric_Pad1.18x1.45mm_HandSolder, F.Cu at (177.5, 96.5)
- added C32: C, Capacitor_SMD:C_0805_2012Metric_Pad1.18x1.45mm_HandSolder, F.Cu at (172.7, 93.5)
- added F1: 20mA, Fuse:Fuse_0805_2012Metric, F.Cu at (157.0, 103.1)
- added J2: Screw_Terminal_01x04, TerminalBlock_Phoenix:TerminalBlock_Phoenix_MPT-0,5-4-2.54_1x04_P2.54mm_Horizontal, F.Cu at (143.0, 84.9)
- added J3: Screw_Terminal_01x04, TerminalBlock_Phoenix:TerminalBlock_Phoenix_MPT-0,5-4-2.54_1x04_P2.54mm_Horizontal, F.Cu at (167.7, 66.6)
- added R27: 100, Resistor_SMD:R_0805_2012Metric_Pad1.20x1.40mm_HandSolder, F.Cu at (180.8, 72.8)
- added R28: 100, Resistor_SMD:R_0805_2012Metric_Pad1.20x1.40mm_HandSolder, F.Cu at (151.2, 99.5)
- added R29: 100, Resistor_SMD:R_0805_2012Metric_Pad1.20x1.40mm_HandSolder, F.Cu at (180.3, 66.9)
- added R30: 100, Resistor_SMD:R_0805_2012Metric_Pad1.20x1.40mm_HandSolder, F.Cu at (185.5, 72.8)
- added R31: 100, Resistor_SMD:R_0805_2012Metric_Pad1.20x1.40mm_HandSolder, F.Cu at (194.6, 63.9)
- added R32: 100, Resistor_SMD:R_0805_2012Metric_Pad1.20x1.40mm_HandSolder, F.Cu at (161.7, 94.3)
- added R33: 0, Resistor_SMD:R_0805_2012Metric_Pad1.20x1.40mm_HandSolder, F.Cu at (189.9, 63.9)
- added R34: 0, Resistor_SMD:R_0805_2012Metric_Pad1.20x1.40mm_HandSolder, F.Cu at (147.7, 102.5)
- added R35: 0, Resistor_SMD:R_0805_2012Metric_Pad1.20x1.40mm_HandSolder, F.Cu at (180.8, 75.8)
- added R36: 0, Resistor_SMD:R_0805_2012Metric_Pad1.20x1.40mm_HandSolder, F.Cu at (189.9, 66.9)
- added U5: MCP3564, Library:MCP3564, F.Cu at (130.7, 93.4)
- C1, C10, C11, C12, C13, C14, C15, C16, C17, C18, C19, C2, C20, C21, C22, C23, C24, C3, C4, C5, C6, C7, C8, C9: footprint Capacitor_SMD:C_0402_1005Metric_Pad0.74x0.62mm_HandSolder -> Capacitor_SMD:C_0805_2012Metric_Pad1.18x1.45mm_HandSolder
- J1: footprint TerminalBlock_TE-Connectivity:TerminalBlock_TE_282834-8_1x08_P2.54mm_Horizontal -> TerminalBlock_Phoenix:TerminalBlock_Phoenix_MPT-0,5-8-2.54_1x08_P2.54mm_Horizontal
- R1, R10, R11, R12, R13, R14, R15, R16, R17, R18, R19, R2, R20, R21, R22, R23, R24, R3, R4, R5, R6, R7, R8, R9: footprint Resistor_SMD:R_0402_1005Metric_Pad0.72x0.64mm_HandSolder -> Resistor_SMD:R_0805_2012Metric_Pad1.20x1.40mm_HandSolder
- R25, R26: value 3k -> 100; footprint Resistor_SMD:R_0402_1005Metric_Pad0.72x0.64mm_HandSolder -> Resistor_SMD:R_0805_2012Metric_Pad1.20x1.40mm_HandSolder
- U4: value LTC2428CGTR -> MCP1501-33xSN; footprint Library:SSOP-28_G -> Package_SO:SOIC-8_3.9x4.9mm_P1.27mm
- moved R21 101.3 mm to (185.0, 66.9)
- moved RV1 99.9 mm to (159.8, 82.6)
- moved R7 99.7 mm to (190.3, 69.8)
- moved R8 98.3 mm to (185.5, 69.9)
- moved R11 97.4 mm to (178.1, 81.0)
- moved R23 89.3 mm to (173.4, 82.4)
- moved R9 88.7 mm to (176.0, 78.1)
- moved R6 87.3 mm to (169.9, 88.3)
- moved R26 85.4 mm to (176.0, 72.2)
- moved R15 85.0 mm to (165.1, 85.4)
- moved R2 84.7 mm to (166.4, 94.2)
- moved R22 81.4 mm to (168.6, 82.4)
- moved R14 79.5 mm to (157.2, 100.2)
- moved R17 78.4 mm to (156.9, 91.3)
- moved C17 78.1 mm to (180.3, 64.0)
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Connections:
- C21 pad 2: unconnected-(C21-Pad2) -> GNDA
- R25 pad 1: +3V3 -> Net-(R25-Pad1)
- R25 pad 2: Net-(R25-Pad2) -> unconnected-(R25-Pad2)
- R26 pad 1: Net-(R25-Pad2) -> Net-(R26-Pad1)
- R26 pad 2: GNDD -> unconnected-(R26-Pad2)
- R5 pad 1: unconnected-(R5-Pad1) -> GNDA
- RV1 pad 1: +3V3 -> ADC_AVDD
- RV1 pad 2: /FSSET -> Net-(U5-Pad3)
- RV1 pad 3: GNDD -> GNDA
- RV2 pad 1: +3V3 -> ADC_AVDD
- RV2 pad 2: /ZSSET -> Net-(C25-Pad1)
- RV2 pad 3: GNDD -> GNDA
- U1 pad 0.20: unconnected-(U1-Pad0.20) -> EN_SENSOR
- U1 pad 0.22: unconnected-(U1-Pad0.22) -> Net-(R25-Pad1)
- U1 pad 0.24: unconnected-(U1-Pad0.24) -> Net-(R26-Pad1)
- U1 pad 0.29: unconnected-(U1-Pad0.29) -> Net-(R27-Pad1)
- U1 pad 0.31: unconnected-(U1-Pad0.31) -> Net-(R28-Pad1)
- U1 pad 1.00: unconnected-(U1-Pad1.00) -> Net-(R29-Pad1)
- U1 pad 1.10: unconnected-(U1-Pad1.10) -> Net-(R30-Pad1)
- U1 pad 1.13: unconnected-(U1-Pad1.13) -> Net-(R31-Pad1)
- U1 pad 1.15: unconnected-(U1-Pad1.15) -> Net-(R32-Pad1)
- U1 pad G1: Net-(U1-PadG1) -> GNDA
- U1 pad G2: Net-(U1-PadG1) -> GNDA
- U1 pad G3: Net-(U1-PadG1) -> GNDA
- U1 pad OUT: unconnected-(U1-PadOUT) -> V_REGOUT0
- U1 pad VBUS: unconnected-(U1-PadVBUS) -> +5V
- U2 pad 4: +5VA -> ADC_AVDD
- U3 pad 10: unconnected-(U3-Pad10) -> GNDA
- U3 pad 4: +5VA -> ADC_AVDD
- U4 pad 1: GNDD -> +5V
- U4 pad 2: +3V3 -> GNDA
- U4 pad 3: /FSSET -> +5V
- U4 pad 4: Net-(U4-Pad4) -> GNDA
- U4 pad 5: /ZSSET -> GNDA
- U4 pad 6: GNDD -> GNDA
- U4 pad 7: Net-(U4-Pad4) -> Net-(U4-Pad7)
- U4 pad 8: +3V3 -> Net-(U4-Pad7)

Commit message: update
Parts:
- removed F1: 20mA, Fuse:Fuse_0805_2012Metric
- added C33: 1uF, Capacitor_SMD:C_0603_1608Metric, F.Cu at (112.8, 136.1)
- added C34: 1uF, Capacitor_SMD:C_0603_1608Metric, F.Cu at (115.6, 133.6)
- added C35: 1uF, Capacitor_SMD:C_0603_1608Metric, F.Cu at (154.9, 99.1)
- added C36: 1uF, Capacitor_SMD:C_0603_1608Metric, F.Cu at (158.0, 96.5)
- added C37: 1uF, Capacitor_SMD:C_0603_1608Metric, F.Cu at (194.6, 69.6)
- added C38: 10µF, Capacitor_SMD:C_0603_1608Metric, F.Cu at (196.1, 130.6)
- added C39: 1uF, Capacitor_SMD:C_0603_1608Metric, F.Cu at (191.5, 72.6)
- added C40: 10µF, Capacitor_SMD:C_0603_1608Metric, F.Cu at (208.3, 130.6)
- added R37: 10, Resistor_SMD:R_0603_1608Metric, F.Cu at (123.2, 127.8)
- added R38: 10, Resistor_SMD:R_0603_1608Metric, F.Cu at (123.2, 140.0)
- added R39: 100, Resistor_SMD:R_0603_1608Metric, F.Cu at (192.3, 134.4)
- added R40: 10, Resistor_SMD:R_0603_1608Metric, F.Cu at (193.8, 129.8)
- added R41: 10k, Resistor_SMD:R_0603_1608Metric, F.Cu at (153.2, 93.5)
- added R42: 10, Resistor_SMD:R_0603_1608Metric, F.Cu at (208.3, 127.5)
- added U6: MCP1754S-5002xCB, Package_TO_SOT_SMD:SOT-23, F.Cu at (112.8, 133.6)
- added U7: MCP1754S-5002xCB, Package_TO_SOT_SMD:SOT-23, F.Cu at (154.9, 96.5)
- added U8: MCP1754S-3302xCB, Package_TO_SOT_SMD:SOT-23, F.Cu at (194.3, 72.4)
- C1, C10, C11, C12, C13, C14, C15, C16, C17, C18, C19, C2, C20, C21, C22, C23, C24, C25, C28, C29, C3, C30, C4, C5, C6, C7, C8, C9: footprint Capacitor_SMD:C_0805_2012Metric_Pad1.18x1.45mm_HandSolder -> Capacitor_SMD:C_0603_1608Metric
- C26: value C -> 2.2µF; footprint Capacitor_SMD:C_0805_2012Metric_Pad1.18x1.45mm_HandSolder -> Capacitor_SMD:C_0603_1608Metric
- C27: value C -> 300pF; footprint Capacitor_SMD:C_0805_2012Metric_Pad1.18x1.45mm_HandSolder -> Capacitor_SMD:C_0603_1608Metric
- C31, C32: value C -> 0.1µF; footprint Capacitor_SMD:C_0805_2012Metric_Pad1.18x1.45mm_HandSolder -> Capacitor_SMD:C_0603_1608Metric
- R1, R10, R11, R12, R13, R14, R15, R16, R17, R18, R19, R2, R20, R21, R22, R23, R24, R25, R26, R27, R28, R29, R3, R30, R31, R32, R33, R34, R35, R36, R4, R5, R6, R7, R8, R9: footprint Resistor_SMD:R_0805_2012Metric_Pad1.20x1.40mm_HandSolder -> Resistor_SMD:R_0603_1608Metric
- moved R7 96.0 mm to (123.2, 138.4), turned to 180 degrees
- moved R21 89.6 mm to (138.9, 143.8), turned to -90 degrees
- moved R8 84.2 mm to (136.7, 138.4)
- moved U5 83.1 mm to (203.2, 134.0)
- moved RV2 83.0 mm to (200.4, 147.3), turned to 180 degrees
- moved C17 78.5 mm to (140.5, 131.6), turned to -90 degrees
- moved R22 77.7 mm to (120.9, 143.8), turned to -90 degrees
- moved C4 77.1 mm to (139.7, 126.2), turned to 180 degrees
- moved R23 75.1 mm to (120.9, 136.1), turned to 90 degrees
- moved R19 73.7 mm to (120.9, 124.0), turned to 90 degrees
- moved U4 72.2 mm to (186.6, 134.6)
- moved RV1 71.9 mm to (200.4, 141.9), turned to 180 degrees
- moved R4 71.6 mm to (136.7, 126.2)
- moved R36 70.8 mm to (195.3, 137.4), turned to 180 degrees
- moved R33 70.7 mm to (195.3, 134.4)
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Connections:
- net Net-(C25-Pad1) renamed REFIN+
- net Net-(U5-Pad3) renamed REFIN-
- C17 pad 2: GNDA -> GND
- C18 pad 2: GNDA -> GND
- C19 pad 2: GNDA -> GND
- C20 pad 2: GNDA -> GND
- C21 pad 2: GNDA -> GND
- C22 pad 2: GNDA -> GND
- C23 pad 2: GNDA -> GND
- C24 pad 2: GNDA -> GND
- C25 pad 2: GNDA -> GND
- C26 pad 1: +5V -> PWR_MAX16V
- C26 pad 2: GNDA -> GND
- C27 pad 1: Net-(U4-Pad7) -> ADC_VREF
- C27 pad 2: GNDA -> GND
- C28 pad 1: +5V -> Net-(C28-Pad1)
- C28 pad 2: GNDA -> GND
- C29 pad 1: ADC_AVDD -> Net-(C29-Pad1)
- C29 pad 2: GNDA -> GND
- C30 pad 1: ADC_AVDD -> Net-(C30-Pad1)
- C30 pad 2: GNDA -> GND
- C31 pad 1: ADC_AVDD -> AVDD
- C31 pad 2: GNDA -> GND
- C32 pad 1: V_REGOUT0 -> DVDD
- C32 pad 2: GNDA -> GND
- J2 pad 1: GNDA -> GND
- J2 pad 2: GNDA -> GND
- J2 pad 3: GNDA -> GND
- J2 pad 4: ADC_AVDD -> GND
- J3 pad 1: GNDA -> GND
- J3 pad 2: GNDA -> GND
- J3 pad 3: GNDA -> GND
- J3 pad 4: +5V -> PWR_MAX16V
- R1 pad 1: GNDA -> GND
- R2 pad 1: GNDA -> GND
- R3 pad 1: GNDA -> GND
- R33 pad 1: ADC_AVDD -> ADC_VREF
- R34 pad 2: GNDA -> GND
- R35 pad 1: ADC_AVDD -> ADC_VREF
- R36 pad 2: GNDA -> GND
- R4 pad 1: GNDA -> GND
- R5 pad 1: GNDA -> GND
- R6 pad 1: GNDA -> GND
- R7 pad 1: GNDA -> GND
- R8 pad 1: GNDA -> GND
- RV1 pad 1: ADC_AVDD -> ADC_VREF
- RV1 pad 3: GNDA -> GND
- RV2 pad 1: ADC_AVDD -> ADC_VREF
- RV2 pad 3: GNDA -> GND
- U1 pad G1: GNDA -> GND
- U1 pad G2: GNDA -> GND
- U1 pad G3: GNDA -> GND
- U1 pad VBUS: +5V -> Net-(C28-Pad1)
- U2 pad 10: GNDA -> GND
- U2 pad 11: GNDA -> GND
- U2 pad 12: GNDA -> GND
- U2 pad 3: GNDA -> GND
- U2 pad 4: ADC_AVDD -> Net-(C29-Pad1)
- U2 pad 5: GNDA -> GND
- U3 pad 10: GNDA -> GND
- U3 pad 11: GNDA -> GND
- U3 pad 12: GNDA -> GND
- U3 pad 3: GNDA -> GND
- U3 pad 4: ADC_AVDD -> Net-(C30-Pad1)
- U3 pad 5: GNDA -> GND
- U4 pad 1: +5V -> PWR_MAX16V
- U4 pad 2: GNDA -> GND
- U4 pad 3: +5V -> PWR_MAX16V
- U4 pad 4: GNDA -> GND
- U4 pad 5: GNDA -> GND
- U4 pad 6: GNDA -> GND
- U5 pad 1: ADC_AVDD -> AVDD
- U5 pad 19: GNDA -> GND
- U5 pad 2: GNDA -> GND
- U5 pad 20: V_REGOUT0 -> DVDD
Routing:
- net GND: track 0.00 -> 106.4 mm
- net Net-(C34-Pad1): track 0.00 -> 25.5 mm
- net ADC_VREF: track 0.00 -> 23.7 mm
- net REFIN+: track 0.00 -> 20.2 mm
- net REFIN-: track 0.00 -> 15.0 mm
- net PWR_MAX16V: track 0.00 -> 14.6 mm
- net Net-(C14-Pad1): track 0.00 -> 10.4 mm
- net Net-(C10-Pad1): track 0.00 -> 10.2 mm
- net Net-(C11-Pad1): track 0.00 -> 8.92 mm
- net Net-(C15-Pad1): track 0.00 -> 8.74 mm
- net Net-(C12-Pad1): track 0.00 -> 7.65 mm
- net Net-(C13-Pad1): track 0.00 -> 7.63 mm
- net Net-(C11-Pad2): track 0.00 -> 7.62 mm
- net Net-(C16-Pad1): track 0.00 -> 7.47 mm
- net Net-(C1-Pad2): track 0.00 -> 7.45 mm
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Other:
- board outline added: 159 x 104.6 mm

Commit message: update
Parts:
- removed C25: C, Capacitor_SMD:C_0603_1608Metric
- removed RV1, RV2: R_Potentiometer_Trim, Potentiometer_THT:Potentiometer_Bourns_3266W_Vertical
- added R43: 10k, Resistor_SMD:R_0603_1608Metric, F.Cu at (130.6, 152.7)
- added R44: 10k, Resistor_SMD:R_0603_1608Metric, F.Cu at (122.7, 147.8)
- added R45: 10k, Resistor_SMD:R_0603_1608Metric, F.Cu at (122.7, 143.3)
- added R46: 10k, Resistor_SMD:R_0603_1608Metric, F.Cu at (130.6, 138.4)
- R1, R2, R3, R4, R5, R6, R7, R8: value 1M -> 10k
- R33, R34, R35, R36: value 0 -> 10k
- moved R35 73.4 mm to (122.7, 125.7), turned to 180 degrees
- moved R34 72.7 mm to (122.7, 130.3)
- moved R36 66.8 mm to (130.6, 120.9)
- moved R33 64.8 mm to (130.6, 135.1), turned to 180 degrees
- moved R5 11.4 mm to (130.6, 151.1)
- moved C6 7.89 mm to (121.2, 149.4)
- moved C30 7.64 mm to (122.7, 146.3), turned to 180 degrees
- moved R1 7.47 mm to (130.6, 133.6)
- moved R4 7.19 mm to (130.6, 122.4)
- moved C22 6.67 mm to (117.3, 150.1)
- moved R22 6.67 mm to (118.9, 150.1)
- moved C5 6.48 mm to (138.4, 147.8)
- moved C14 6.43 mm to (125.0, 150.1)
- moved R14 6.43 mm to (123.4, 150.1)
- moved C13 6.36 mm to (136.1, 150.1)
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Connections:
- net /OUT0 renamed /ADC_CH0
- net /OUT1 renamed /ADC_CH1
- net /OUT2 renamed /ADC_CH2
- net /OUT3 renamed /ADC_CH3
- net /OUT4 renamed /ADC_CH4
- net /OUT5 renamed /ADC_CH5
- net /OUT6 renamed /ADC_CH6
- net /OUT7 renamed /ADC_CH7
- net AVDD renamed ADC_AVDD
- net Net-(C28-Pad1) renamed NRF_VBUS
- net Net-(C34-Pad1) renamed TIA_V
- C27 pad 1: ADC_VREF -> ADC_VREF+
- C29 pad 1: Net-(C29-Pad1) -> TIA0_V
- C30 pad 1: Net-(C30-Pad1) -> TIA1_V
- C32 pad 1: DVDD -> ADC_DVDD
- C40 pad 1: DVDD -> ADC_DVDD
- R1 pad 1: GND -> TIA0_V
- R1 pad 2: Net-(C1-Pad2) -> Net-(U2-Pad10)
- R2 pad 1: GND -> TIA0_V
- R2 pad 2: Net-(C10-Pad1) -> Net-(U2-Pad5)
- R3 pad 1: GND -> TIA0_V
- R3 pad 2: Net-(C11-Pad1) -> Net-(U2-Pad3)
- R33 pad 1: ADC_VREF -> Net-(U2-Pad10)
- R33 pad 2: REFIN- -> GND
- R34 pad 1: REFIN- -> Net-(U2-Pad5)
- R35 pad 1: ADC_VREF -> Net-(U2-Pad3)
- R35 pad 2: REFIN+ -> GND
- R36 pad 1: REFIN+ -> Net-(U2-Pad12)
- R37 pad 2: Net-(C29-Pad1) -> TIA0_V
- R38 pad 2: Net-(C30-Pad1) -> TIA1_V
- R39 pad 2: ADC_VREF -> ADC_VREF+
- R4 pad 1: GND -> TIA0_V
- R4 pad 2: Net-(C12-Pad1) -> Net-(U2-Pad12)
- R41 pad 1: V_REGOUT0 -> ADC_DVDD
- R42 pad 1: DVDD -> ADC_DVDD
- R42 pad 2: V_REGOUT0 -> NRF_REG0_V
- R5 pad 1: GND -> TIA1_V
- R5 pad 2: Net-(C13-Pad1) -> Net-(U3-Pad10)
- R6 pad 1: GND -> TIA1_V
- R6 pad 2: Net-(C14-Pad1) -> Net-(U3-Pad5)
- R7 pad 1: GND -> TIA1_V
- R7 pad 2: Net-(C15-Pad1) -> Net-(U3-Pad3)
- R8 pad 1: GND -> TIA1_V
- R8 pad 2: Net-(C16-Pad1) -> Net-(U3-Pad12)
- U1 pad 0.20: EN_SENSOR -> unconnected-(U1-Pad0.20)
- U1 pad OUT: V_REGOUT0 -> NRF_REG0_V
- U2 pad 10: GND -> Net-(U2-Pad10)
- U2 pad 12: GND -> Net-(U2-Pad12)
- U2 pad 3: GND -> Net-(U2-Pad3)
- U2 pad 4: Net-(C29-Pad1) -> TIA0_V
- U2 pad 5: GND -> Net-(U2-Pad5)
- U3 pad 10: GND -> Net-(U3-Pad10)
- U3 pad 12: GND -> Net-(U3-Pad12)
- U3 pad 3: GND -> Net-(U3-Pad3)
- U3 pad 4: Net-(C30-Pad1) -> TIA1_V
- U3 pad 5: GND -> Net-(U3-Pad5)
- U5 pad 20: DVDD -> ADC_DVDD
- U5 pad 3: REFIN- -> GND
- U5 pad 4: REFIN+ -> ADC_VREF+
Routing:
- net GND: track 106.4 -> 36.0 mm, vias 0 -> 16
- net /CH4: track 0.00 -> 61.6 mm
- net /CH3: track 0.00 -> 60.4 mm
- net /CH7: track 0.00 -> 33.9 mm
- net /CH0: track 0.00 -> 32.0 mm
- net TIA0_V: track 0.00 -> 24.0 mm
- net TIA1_V: track 0.00 -> 24.0 mm
- net ADC_VREF: track 23.7 -> 0.00 mm
- net REFIN+: track 20.2 -> 0.00 mm
- net /CH1: track 0.00 -> 19.5 mm, vias 0 -> 1
- net /CH6: track 0.00 -> 19.4 mm, vias 0 -> 1
- net REFIN-: track 15.0 -> 0.00 mm
- net PWR_MAX16V: track 14.6 -> 0.00 mm
- net Net-(U2-Pad12): track 0.00 -> 7.38 mm
- net Net-(U2-Pad10): track 0.00 -> 7.38 mm
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- added copper zone on B.Cu, net GND
Other:
- board size 159 x 104.6 mm -> 159 x 111.5 mm

Commit message: update
Parts:
- added J4: Conn_01x08_Female, Connector_PinSocket_2.54mm:PinSocket_1x08_P2.54mm_Vertical, F.Cu at (153.2, 126.7)
