File: circuit1/namp.kicad_pcb (KiCad board)
At the start: 2 copper layers, 159 x 111.5 mm, 97 parts, among them J1 Screw_Terminal_01x08, J2 Screw_Terminal_01x04, J3 Screw_Terminal_01x04, J4 Conn_01x08_Female, U1 NRF52840-DONGLE, U2 MCP6004, U3 MCP6004, U4 MCP1501-33xSN, U5 MCP3564, U6 MCP1754S-5002xCB, U7 MCP1754S-5002xCB, U8 MCP1754S-3302xCB

Commit message: update
Parts:
- J4: footprint Connector_PinSocket_2.54mm:PinSocket_1x08_P2.54mm_Vertical -> Connector_PinHeader_2.54mm:PinHeader_1x08_P2.54mm_Vertical
- moved R42 36.7 mm to (171.7, 130.7)
- moved U5 36.7 mm to (166.6, 137.2)
- moved C32 36.7 mm to (173.2, 133.6)
- moved C40 36.7 mm to (171.7, 133.6)
- moved C31 36.5 mm to (161.3, 133.7)
- moved C38 36.5 mm to (159.8, 133.7)
- moved R40 33.3 mm to (160.5, 131.6), turned to 0 degrees
- moved R39 27.8 mm to (165.9, 142.9), turned to 90 degrees
- moved C26 26.6 mm to (164.6, 153.4), turned to 0 degrees
- moved C27 25.9 mm to (167.4, 142.9), turned to -90 degrees
- moved U4 24.8 mm to (166.1, 148.6), turned to 90 degrees
- moved C22 3.81 mm to (120.4, 152.4), turned to 90 degrees
- moved R22 3.81 mm to (121.9, 152.4), turned to 90 degrees
- moved J4 3.62 mm to (149.9, 128.3)
- moved C18 3.41 mm to (120.4, 134.1), turned to 90 degrees
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Connections:
- C1 pad 1: /CH0 -> /CH2
- C17 pad 1: /ADC_CH0 -> /ADC_CH2
- C18 pad 1: /ADC_CH1 -> /ADC_CH3
- C19 pad 1: /ADC_CH2 -> /ADC_CH0
- C2 pad 1: /CH1 -> /CH3
- C20 pad 1: /ADC_CH3 -> /ADC_CH1
- C21 pad 1: /ADC_CH4 -> /ADC_CH6
- C22 pad 1: /ADC_CH5 -> /ADC_CH7
- C23 pad 1: /ADC_CH6 -> /ADC_CH4
- C24 pad 1: /ADC_CH7 -> /ADC_CH5
- C3 pad 1: /CH2 -> /CH0
- C4 pad 1: /CH3 -> /CH1
- C5 pad 1: /CH4 -> /CH6
- C6 pad 1: /CH5 -> /CH7
- C7 pad 1: /CH6 -> /CH4
- C8 pad 1: /CH7 -> /CH5
- R17 pad 1: /ADC_CH0 -> /ADC_CH2
- R18 pad 1: /ADC_CH1 -> /ADC_CH3
- R19 pad 1: /ADC_CH2 -> /ADC_CH0
- R20 pad 1: /ADC_CH3 -> /ADC_CH1
- R21 pad 1: /ADC_CH4 -> /ADC_CH6
- R22 pad 1: /ADC_CH5 -> /ADC_CH7
- R23 pad 1: /ADC_CH6 -> /ADC_CH4
- R24 pad 1: /ADC_CH7 -> /ADC_CH5
Routing:
- net /ADC_CH7: track 1.54 -> 66.7 mm, vias 0 -> 1
- net /ADC_CH0: track 1.54 -> 56.0 mm
- net /ADC_CH3: track 1.54 -> 45.6 mm
- net /ADC_CH4: track 1.54 -> 44.8 mm
- net /CH5: track 0.00 -> 40.8 mm, vias 0 -> 1
- net /CH4: track 61.6 -> 21.1 mm, vias 0 -> 1
- net /CH2: track 0.00 -> 40.4 mm, vias 0 -> 1
- net /CH3: track 60.4 -> 21.0 mm, vias 0 -> 1
- net /ADC_CH6: track 1.54 -> 40.9 mm, vias 0 -> 1
- net GND: track 36.0 -> 71.1 mm, vias 16 -> 21
- net /ADC_CH1: track 1.54 -> 32.0 mm
- net /ADC_CH2: track 1.54 -> 27.2 mm
- net /ADC_CH5: track 1.54 -> 25.6 mm
- net /CH1: track 19.5 -> 40.9 mm
- net /CH6: track 19.4 -> 40.6 mm
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