File: circuit2/namp.kicad_pcb (KiCad board)
At the start: 2 copper layers, 90 x 75 mm, 97 parts, among them J1 Screw_Terminal_01x08, J2 Screw_Terminal_01x04, J3 Screw_Terminal_01x04, J4 Conn_01x08_Female, J5 Conn_01x08_Male, U1 NRF52840-DONGLE, U2 MCP6004, U3 MCP6004, U4 MCP1501-33xSN, U5 MCP3564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

Commit message: update
Parts:
- removed R26: 10, Resistor_SMD:R_0805_2012Metric_Pad1.20x1.40mm_HandSolder
- removed R39: 100, Resistor_SMD:R_0805_2012Metric_Pad1.20x1.40mm_HandSolder
- removed REF**: MountingHole_3.2mm_M3, MountingHole:MountingHole_3.2mm_M3
- added C36: 0.1µF, Capacitor_SMD:C_0805_2012Metric_Pad1.18x1.45mm_HandSolder, F.Cu at (163.3, 151.4)
- C26: value 2.2µF -> 0.1µF
- C27: value 300pF -> 0.1µF
- U4: value MCP1501-33xSN -> MAX6070; footprint Package_SO:SOIC-8_3.9x4.9mm_P1.27mm -> Package_TO_SOT_SMD:SOT-23-6_Handsoldering
- moved C26 4.00 mm to (168.0, 151.4), turned to 180 degrees
- moved C28 3.24 mm to (162.7, 109.0), turned to -90 degrees
- moved U4 2.16 mm to (165.7, 147.1)
- moved C25 1.96 mm to (111.0, 107.2), turned to -90 degrees
- moved C27 1.53 mm to (166.4, 143.1), turned to 0 degrees
Connections:
- C26 pad 1: Net-(C26-Pad1) -> TIA_4.5V
- U4 pad 1: Net-(C26-Pad1) -> Net-(C36-Pad1)
- U4 pad 3: Net-(C26-Pad1) -> TIA_4.5V
- U4 pad 4: GND -> TIA_4.5V
- U4 pad 5: GND -> ADC_VREF+
- U4 pad 6: GND -> ADC_VREF+
Routing:
- net +5V: track 247.9 -> 155.7 mm
- net TIA_4.5V: track 33.6 -> 122.0 mm
- net Net-(C26-Pad1): track 12.4 -> 0.00 mm
- net GND: track 98.8 -> 106.1 mm, vias 38 -> 34
- net Net-(R39-Pad1): track 5.13 -> 0.00 mm
- net Net-(C36-Pad1): track 0.00 -> 4.61 mm
- net ADC_VREF+: track 9.98 -> 13.9 mm
- net PWR_MAX15V: track 17.6 -> 14.4 mm
- removed copper zone on F.Cu, net GND

Commit message: update
Parts:
- added C41: 10nF, Capacitor_SMD:C_0805_2012Metric_Pad1.18x1.45mm_HandSolder, F.Cu at (156.3, 127.4)
- C38: value 10µF -> 0.1µF
- C39: value 1uF -> 2.2uF
- C40: value 10µF -> 0.1uF
- U8: value LP5907MFX-3.3 -> LP2985-3.6
- moved C28 1.77 mm to (163.1, 110.7), turned to 0 degrees
Connections:
- U8 pad 4: unconnected-(U8-Pad4) -> Net-(C41-Pad1)
Routing:
- net GND: track 106.1 -> 80.2 mm, vias 34 -> 30
- net +5V: track 155.7 -> 158.3 mm
- net Net-(C41-Pad1): track 0.00 -> 2.49 mm
- net NRF_REG0_V: track 30.9 -> 30.1 mm
- added copper zone on F.Cu, net GND
Other:
- board text added: "3.3V VREF"
- board text added: "3.6V VREG"
- board text added: "4.5V VREG"
- board text added: "5V VREG"

Commit message: update
Parts:
- U2, U3: value MCP6004 -> MCP6034
- moved C25 0.25 mm to (111.3, 107.2)
Routing:
- net GND: track 80.2 -> 69.0 mm
Changed lines of the file:
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@@
   (net 57 "ADC_MCK")
   (net 58 "Net-(R25-Pad1)")
-  (net 59 "Net-(R40-Pad2)")
+  (net 59 "Net-(C39-Pad1)")
   (net 60 "/ADC_CH0")
   (net 61 "Net-(R1-Pad2)")
@@
       (effects (font (size 1 1) (thickness 0.15)))
     )
-    (fp_text value "MCP6004" (at 0 5.28) (layer "F.Fab")
+    (fp_text value "MCP6034" (at 0 5.28) (layer "F.Fab")
       (effects (font (size 1 1) (thickness 0.15)))
     )
@@
       (net 55 "ADC_AVDD") (pintype "passive"))
     (pad "2" smd roundrect (at 1 0) (size 1.2 1.4) (layers "F.Cu" "F.Paste" "F.Mask") (roundrect_rratio 0.208333)
-      (net 59 "Net-(R40-Pad2)") (pintype "passive"))
+      (net 59 "Net-(C39-Pad1)") (pintype "passive"))
     (model "${KICAD6_3DMODEL_DIR}/Resistor_SMD.3dshapes/R_0805_2012Metric.wrl"
       (offset (xyz 0 0 0))
@@
   )
   (footprint "Capacitor_THT:CP_Radial_D5.0mm_P2.00mm" (layer "F.Cu")
-    (at 110.998 107.248888 -90)
+    (at 111.252 107.248888 -90)
     (descr "CP, Radial series, Radial, pin pitch=2.00mm, , diameter=5mm, Electrolytic Capacitor")
     (tags "CP Radial series Radial pin pitch 2.00mm  diameter 5mm Electrolytic Capacitor")
@@
       (net 76 "Net-(C41-Pad1)") (pinfunction "BP") (pintype "input"))
     (pad "5" smd roundrect (at 1.1375 -0.95 270) (size 1.325 0.6) (layers "F.Cu" "F.Paste" "F.Mask") (roundrect_rratio 0.25)
-      (net 59 "Net-(R40-Pad2)") (pinfunction "VOUT") (pintype "power_out"))
+      (net 59 "Net-(C39-Pad1)") (pinfunction "VOUT") (pintype "power_out"))
     (model "${KICAD6_3DMODEL_DIR}/Package_TO_SOT_SMD.3dshapes/SOT-23-5.wrl"
       (offset (xyz 0 0 0))
@@
     (fp_line (start 1 0.625) (end -1 0.625) (layer "F.Fab") (width 0.1))
     (pad "1" smd roundrect (at -1.0375 0 180) (size 1.175 1.45) (layers "F.Cu" "F.Paste" "F.Mask") (roundrect_rratio 0.212766)
-      (net 59 "Net-(R40-Pad2)") (pintype "passive"))
+      (net 59 "Net-(C39-Pad1)") (pintype "passive"))
     (pad "2" smd roundrect (at 1.0375 0 180) (size 1.175 1.45) (layers "F.Cu" "F.Paste" "F.Mask") (roundrect_rratio 0.212766)
       (net 25 "GND") (pintype "passive"))
@@
       (effects (font (size 1 1) (thickness 0.15)))
     )
-    (fp_text value "MCP6004" (at 0 5.28) (layer "F.Fab")
+    (fp_text value "MCP6034" (at 0 5.28) (layer "F.Fab")
       (effects (font (size 1 1) (thickness 0.15)))
     )
@@
   (segment (start 129.556 133.858) (end 127.762 133.858) (width 0.5) (layer "F.Cu") (net 25))
   (segment (start 171.460499 134.885001) (end 172.466 133.8795) (width 0.3) (layer "F.Cu") (net 25))
-  (segment (start 102.117 98.538) (end 101.854 98.801) (width 1) (layer "F.Cu") (net 25))
   (segment (start 168.275 143.129) (end 168.91 143.764) (width 0.5) (layer "F.Cu") (net 25))
-  (segment (start 112.928 98.538) (end 102.117 98.538) (width 1) (layer "F.Cu") (net 25))
   (segment (start 110.236 135.1495) (end 109.1985 134.112) (width 0.5) (layer "F.Cu") (net 25))
   (segment (start 143.002 120.1205) (end 143.002 118.364) (width 0.5) (layer "F.Cu") (net 25))

Commit message: Added holes
Parts:
- added REF**: MountingHole_3.2mm_M3, MountingHole:MountingHole_3.2mm_M3, F.Cu at (181.5, 157.6)
- added REF**: MountingHole_3.2mm_M3, MountingHole:MountingHole_3.2mm_M3, F.Cu at (181.5, 92.6)
- added REF**: MountingHole_3.2mm_M3, MountingHole:MountingHole_3.2mm_M3, F.Cu at (101.5, 92.6)
- added REF**: MountingHole_3.2mm_M3, MountingHole:MountingHole_3.2mm_M3, F.Cu at (101.5, 157.6)
Changed lines of the file:
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@@
     )
+  )
+  (footprint "MountingHole:MountingHole_3.2mm_M3" (layer "F.Cu")
+    (at 181.52 157.56)
+    (descr "Mounting Hole 3.2mm, no annular, M3")
+    (tags "mounting hole 3.2mm no annular m3")
+    (attr exclude_from_pos_files exclude_from_bom)
+    (fp_text reference "REF**" (at 0 -4.2) (layer "F.SilkS")
+      (effects (font (size 1 1) (thickness 0.15)))
+    )
+    (fp_text value "MountingHole_3.2mm_M3" (at 0 4.2) (layer "F.Fab")
+      (effects (font (size 1 1) (thickness 0.15)))
+    )
+    (fp_text user "${REFERENCE}" (at 0.3 0) (layer "F.Fab")
+      (effects (font (size 1 1) (thickness 0.15)))
+    )
+    (fp_circle (center 0 0) (end 3.2 0) (layer "Cmts.User") (width 0.15) (fill none))
+    (fp_circle (center 0 0) (end 3.45 0) (layer "F.CrtYd") (width 0.05) (fill none))
+    (pad "" np_thru_hole circle (at 0 0) (size 3.2 3.2) (drill 3.2) (layers *.Cu *.Mask))
   )
   (footprint "Package_TO_SOT_SMD:SOT-23-5" (layer "F.Cu")
@@
       (rotate (xyz 0 0 0))
     )
+  )
+  (footprint "MountingHole:MountingHole_3.2mm_M3" (layer "F.Cu")
+    (at 181.52 92.56)
+    (descr "Mounting Hole 3.2mm, no annular, M3")
+    (tags "mounting hole 3.2mm no annular m3")
+    (attr exclude_from_pos_files exclude_from_bom)
+    (fp_text reference "REF**" (at 0 -4.2) (layer "F.SilkS")
+      (effects (font (size 1 1) (thickness 0.15)))
+    )
+    (fp_text value "MountingHole_3.2mm_M3" (at 0 4.2) (layer "F.Fab")
+      (effects (font (size 1 1) (thickness 0.15)))
+    )
+    (fp_text user "${REFERENCE}" (at 0.3 0) (layer "F.Fab")
+      (effects (font (size 1 1) (thickness 0.15)))
+    )
+    (fp_circle (center 0 0) (end 3.2 0) (layer "Cmts.User") (width 0.15) (fill none))
+    (fp_circle (center 0 0) (end 3.45 0) (layer "F.CrtYd") (width 0.05) (fill none))
+    (pad "" np_thru_hole circle (at 0 0) (size 3.2 3.2) (drill 3.2) (layers *.Cu *.Mask))
   )
   (footprint "Resistor_SMD:R_0805_2012Metric_Pad1.20x1.40mm_HandSolder" (layer "F.Cu")
@@
       (rotate (xyz 0 0 0))
     )
+  )
+  (footprint "MountingHole:MountingHole_3.2mm_M3" (layer "F.Cu")
+    (at 101.52 92.56)
+    (descr "Mounting Hole 3.2mm, no annular, M3")
+    (tags "mounting hole 3.2mm no annular m3")
+    (attr exclude_from_pos_files exclude_from_bom)
+    (fp_text reference "REF**" (at 0 -4.2) (layer "F.SilkS")
+      (effects (font (size 1 1) (thickness 0.15)))
+    )
+    (fp_text value "MountingHole_3.2mm_M3" (at 0 4.2) (layer "F.Fab")
+      (effects (font (size 1 1) (thickness 0.15)))
+    )
+    (fp_text user "${REFERENCE}" (at 0.3 0) (layer "F.Fab")
+      (effects (font (size 1 1) (thickness 0.15)))
+    )
+    (fp_circle (center 0 0) (end 3.2 0) (layer "Cmts.User") (width 0.15) (fill none))
+    (fp_circle (center 0 0) (end 3.45 0) (layer "F.CrtYd") (width 0.05) (fill none))
+    (pad "" np_thru_hole circle (at 0 0) (size 3.2 3.2) (drill 3.2) (layers *.Cu *.Mask))
   )
   (footprint "Capacitor_SMD:C_0805_2012Metric_Pad1.18x1.45mm_HandSolder" (layer "F.Cu")
@@
     )
   )
+  (footprint "MountingHole:MountingHole_3.2mm_M3" (layer "F.Cu")
+    (at 101.52 157.56)
+    (descr "Mounting Hole 3.2mm, no annular, M3")
+    (tags "mounting hole 3.2mm no annular m3")
+    (attr exclude_from_pos_files exclude_from_bom)
+    (fp_text reference "REF**" (at 0 -4.2) (layer "F.SilkS")
+      (effects (font (size 1 1) (thickness 0.15)))
+    )
+    (fp_text value "MountingHole_3.2mm_M3" (at 0 4.2) (layer "F.Fab")
+      (effects (font (size 1 1) (thickness 0.15)))
+    )
+    (fp_text user "${REFERENCE}" (at 0.3 0) (layer "F.Fab")
+      (effects (font (size 1 1) (thickness 0.15)))
+    )
+    (fp_circle (center 0 0) (end 3.2 0) (layer "Cmts.User") (width 0.15) (fill none))
+    (fp_circle (center 0 0) (end 3.45 0) (layer "F.CrtYd") (width 0.05) (fill none))
+    (pad "" np_thru_hole circle (at 0 0) (size 3.2 3.2) (drill 3.2) (layers *.Cu *.Mask))
+  )
   (footprint "Capacitor_SMD:C_0805_2012Metric_Pad1.18x1.45mm_HandSolder" (layer "F.Cu")

Commit message: update
Routing:
- net /ADC_CH2: track 26.7 -> 27.8 mm
- net ADC_INT: track 53.3 -> 52.4 mm
Other:
- outline, holes or cut-outs redrawn
- board text added: "4.5V"
- board text added: "5V"
- board text added: "5V VREG LM1117"
- board text added: "6.5V-15V"
- board text added: "LP2985"
- board text added: "LP5907"
- board text added: "MAX6070"
- board text added: "MCP3564"
- board text added: "REG0_V"
- board text added: "TIABT V0.1 by RISE An 8 channel TIA ADC Bluetooth"
- board text added: "nRF52840 Dongle"
- board text removed: "5V VREG"
