File: circuit2/namp.kicad_pcb (KiCad board)
At the start: 2 copper layers, 90 x 75 mm, 100 parts, among them J1 Screw_Terminal_01x08, J2 Screw_Terminal_01x04, J3 Screw_Terminal_01x04, J4 Conn_01x08_Female, J5 Conn_01x08_Male, U1 NRF52840-DONGLE, U2 MCP6034, U3 MCP6034, U4 MAX6070, U5 MCP3564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

Commit message: Update
Parts:
- moved C27 2.29 mm to (164.1, 143.1), turned to 180 degrees
- renumbered REF** to M3
Routing:
- net GND: track 69.0 -> 55.0 mm, vias 30 -> 35
- net /ADC_CH2: track 27.8 -> 26.7 mm
- net /ADC_CH0: track 60.3 -> 59.2 mm
Other:
- board text added: "ADC IO"
- board text added: "TIA Output"
- board text added: "TIABT V1 by RISE 2022-02-18 An 8 channel TIA ADC Bluetooth Measurement unit"
- board text removed: "TIABT V0.1 by RISE An 8 channel TIA ADC Bluetooth"

Commit message: update
Parts:
- moved C26 4.66 mm to (168.9, 146.8), turned to -90 degrees
- moved C36 2.17 mm to (162.6, 149.4), turned to -90 degrees
Routing:
- net TIA_4.5V: track 122.0 -> 129.3 mm
- net Net-(C36-Pad1): track 4.61 -> 2.27 mm
- net GND: track 55.0 -> 55.5 mm, vias 35 -> 37
