File: circuit2/namp.kicad_sch (KiCad schematic)
At the start: 96 parts, among them J1 Screw_Terminal_01x08, J2 Screw_Terminal_01x04, J3 Screw_Terminal_01x04, J4 Conn_01x08_Female, J5 Conn_01x08_Male, U1 NRF52840-DONGLE, U2 MCP6004, U3 MCP6004, U4 MCP1501-33xSN, U5 MCP3564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

Commit message: update
Parts:
- removed R26: 10, Resistor_SMD:R_0805_2012Metric_Pad1.20x1.40mm_HandSolder, symbol Device:R
- removed R39: 100, Resistor_SMD:R_0805_2012Metric_Pad1.20x1.40mm_HandSolder, symbol Device:R
- removed U4: MCP1501-33xSN, Package_SO:SOIC-8_3.9x4.9mm_P1.27mm, symbol Reference_Voltage:MCP1501-33xSN
- added C36: 0.1µF, Capacitor_SMD:C_0805_2012Metric_Pad1.18x1.45mm_HandSolder, symbol Device:C
- added U4: MAX6070, Package_TO_SOT_SMD:SOT-23-6_Handsoldering, symbol max6070:MAX6070
- C26: value 2.2µF -> 0.1µF
- C27: value 300pF -> 0.1µF
Connections:
- net ADC_VREF+: now also U4.5 (OUTS), U4.6 (OUTF)
- net GND: now also C36.2, U4.2 (GND)
- net TIA_4.5V: now also C26.1, U4.3 (EN), U4.4 (IN)
- new net: C36.1, U4.1 (FILTER)
Other:
- note added: "Analog Power"
- note added: "Main Power"
- note removed: "Power"
- note removed: "The MCP1501 is a buffered voltage reference capable of sinking and sourcing 20 mA of current. The voltage reference is a low-drift bandgap-based reference. The bandgap uses chopper-based amplifiers, effectively reducing the drift to zero."
- moved on the sheet: C26

Commit message: update
Parts:
- removed U8: LP5907MFX-3.3, Package_TO_SOT_SMD:SOT-23-5, symbol Regulator_Linear:LP5907MFX-3.3
- added C41: 10nF, Capacitor_SMD:C_0805_2012Metric_Pad1.18x1.45mm_HandSolder, symbol Device:C
- added U8: LP2985-3.6, Package_TO_SOT_SMD:SOT-23-5, symbol Regulator_Linear:LP2985-3.3
- C38: value 10µF -> 0.1µF
- C39: value 1uF -> 2.2uF
- C40: value 10µF -> 0.1uF
Connections:
- net +5V: now also U8.1 (VIN), U8.3 (ON/~{OFF})
- net GND: now also C41.2, U8.2 (GND)
- net at C39.1, R40.2: now also U8.5 (VOUT)
- new net: C41.1, U8.4 (BP)
Other:
- moved on the sheet: C37, C39

Commit message: update
Parts:
- U2, U3: value MCP6004 -> MCP6034
Other:
- moved on the sheet: C29, C30, C33, C34, R37, R38, U2E, U3E, U6

Commit message: test
Other:
- note added: "https://www.digikey.se/sv/articles/how-to-design-stable-transimpedance-amplifiers-automotive-medical-systems MCP6034 OpAmp: C_CM = 6pF C_DIFF = 6pF GBWP = 10kHz MOLOKO Photodiode: C_PD = ? , exemple Vishay TEFD4300 is 3.3pF Cin = C_CM + C_DIFF + C_PD = 6+6+3.3 = 15.3pF Cf = sqrt(Cin / (2*PI*Rf*GPWP)) Cf = sqrt((15.3*10^(-12))/(2*pi*(1*10^6) * (10*10^3))) Cf = 1.54509680809275832136877094124595565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"
Changed lines of the file:
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@@
     (effects (font (size 4 4)) (justify left bottom))
+  )
+  (text "https://www.digikey.se/sv/articles/how-to-design-stable-transimpedance-amplifiers-automotive-medical-systems\n\nMCP6034 OpAmp:\nC_CM = 6pF\nC_DIFF = 6pF\nGBWP = 10kHz\n\nMOLOKO Photodiode:\nC_PD = ? , exemple Vishay TEFD4300 is 3.3pF\n\n\n\nCin = C_CM + C_DIFF + C_PD = 6+6+3.3 = 15.3pF\nCf = sqrt(Cin / (2*PI*Rf*GPWP))\nCf = sqrt((15.3*10^(-12))/(2*pi*(1*10^6) * (10*10^3)))\nCf = 1.5450968080927583213687709412459556523443978567508523833347 × 10^-11\nCf = 15pF\n\n\n"
+    (at 132.08 201.93 0)
+    (effects (font (size 1.27 1.27)) (justify left bottom))
   )
   (text "In High Voltage mode, \nthe output from REG0 can be used to \nsupply external circuitry from the VDD pin. \nThe VDD output voltage is \nconfigured in the register REGOUT0 for \n1.8V, 2.1V, 2.4V, 2.7V, 3.0V and 3.3V."

Commit message: addded circuit 3
Parts:
- added J6: RFShield_OnePiece, symbol Device:RFShield_OnePiece
Connections:
- net GND: now also J6.1 (Shield)
Changed lines of the file:
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@@
     (pin "2")
+  )
+  (symbol (lib_id "power:GND") (at 290.83 369.57 0) (unit 1)
+    (in_bom yes) (on_board yes) (fields_autoplaced)
+    (property "Reference" "#PWR?" (id 0) (at 290.83 375.92 0)
+      (effects (font (size 1.27 1.27)) hide)
+    )
+    (property "Value" "GND" (id 1) (at 290.83 374.65 0))
+    (property "Footprint" "" (id 2) (at 290.83 369.57 0)
+      (effects (font (size 1.27 1.27)) hide)
+    )
+    (property "Datasheet" "" (id 3) (at 290.83 369.57 0)
+      (effects (font (size 1.27 1.27)) hide)
+    )
+    (pin "1")
   )
   (symbol (lib_id "Connector:Conn_01x08_Female") (at 236.22 373.38 0) (unit 1)
@@
     (pin "1")
   )
+  (symbol (lib_id "Device:RFShield_OnePiece") (at 290.83 359.41 0) (unit 1)
+    (in_bom yes) (on_board yes) (fields_autoplaced)
+    (property "Reference" "J6" (id 0) (at 307.34 358.1399 0)
+      (effects (font (size 1.27 1.27)) (justify left))
+    )
+    (property "Value" "RFShield_OnePiece" (id 1) (at 307.34 360.6799 0)
+      (effects (font (size 1.27 1.27)) (justify left))
+    )
+    (property "Footprint" "" (id 2) (at 290.83 361.95 0)
+      (effects (font (size 1.27 1.27)) hide)
+    )
+    (property "Datasheet" "~" (id 3) (at 290.83 361.95 0)
+      (effects (font (size 1.27 1.27)) hide)
+    )
+    (pin "1")
+  )
   (symbol (lib_id "Device:C") (at 425.45 264.16 0) (unit 1)
     (in_bom yes) (on_board yes) (fields_autoplaced)
@@
       (reference "#PWR0133") (unit 1) (value "+5V") (footprint "")
     )
+    (path "/549b42ab-db9d-41e6-b6ee-149f2ee2b00b"
+      (reference "#PWR?") (unit 1) (value "GND") (footprint "")
+    )
     (path "/b11c1345-5d6b-4d2f-a711-64752dfa97de"
       (reference "C1") (unit 1) (value "10pF") (footprint "Capacitor_SMD:C_0805_2012Metric_Pad1.18x1.45mm_HandSolder")
@@
       (reference "J5") (unit 1) (value "Conn_01x08_Male") (footprint "Connector_PinHeader_2.54mm:PinHeader_1x08_P2.54mm_Vertical")
     )
+    (path "/ba2a1b2d-a432-436d-b1c0-4f07ac548fa3"
+      (reference "J6") (unit 1) (value "RFShield_OnePiece") (footprint "")
+    )
     (path "/0a4670fe-f411-47c9-8912-2ac7b841eb8f"
