File: circuit3/namp.kicad_sch (KiCad schematic)
At the start: 66 parts, among them J1 Screw_Terminal_01x08, J2 Screw_Terminal_01x04, J3 Screw_Terminal_01x04, J4 Conn_01x08_Female, J5 Conn_01x08_Male, J6 RFShield_OnePiece, U2 MCP6034, U3 MCP6034, U4 MAX6070, U5 MCP3564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

Commit message: update
Parts:
- added U1: Sensor_OPDOLED, Moloko:Sensor_OPDOLED, symbol Moloko:Sensor_OPDOLED
- J6: footprint RF_Shielding:Wuerth_36103505_50x50mm -> RF_Shielding:Wuerth_36503605_60x60mm
Connections:
- net CH0: now also U1.1 (OPD1-)
- net CH1: now also U1.1 (OPD1-)
- net GND: now also U1.0 (OPD1+)
Other:
- note added: "https://www.nwengineeringllc.com/article/should-you-split-ground-planes-in-mixed-signal-pcb-design.php https://electronics.stackexchange.com/questions/22223/shielding-can-what-is-the-proper-way"
