File: circuit3/namp.kicad_pcb (KiCad board)
At the start: 2 copper layers, 90 x 75 mm, 66 parts, among them J1 Screw_Terminal_01x08, J2 Screw_Terminal_01x04, J3 Screw_Terminal_01x04, J4 Conn_01x08_Female, J5 Conn_01x08_Male, J6 RFShield_OnePiece, U2 MCP6034, U3 MCP6034, U4 MAX6070, U5 MCP3564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

Commit message: update
Parts:
- added U1: Sensor_OPDOLED, Moloko:Sensor_OPDOLED, F.Cu at (195.4, 105.7)
- J4: moved to B.Cu
- J6: footprint RF_Shielding:Wuerth_36103505_50x50mm -> RF_Shielding:Wuerth_36503605_60x60mm
- moved J3 28.2 mm to (102.5, 70.6)
- moved C25 28.2 mm to (111.9, 79.1)
- moved C35 28.2 mm to (120.0, 80.0)
- moved U7 28.2 mm to (116.7, 72.6)
- moved C34 24.2 mm to (128.8, 125.4), turned to -90 degrees
- moved U6 19.5 mm to (125.5, 125.4), turned to 0 degrees
- moved C12 16.1 mm to (133.1, 105.4)
- moved C20 16.1 mm to (139.9, 105.4)
- moved R12 16.1 mm to (135.4, 105.4)
- moved R20 16.1 mm to (137.7, 105.4)
- moved U2 16.1 mm to (127.5, 109.9)
- moved C11 16.1 mm to (121.2, 103.1)
- moved C18 16.1 mm to (114.5, 118.8)
- moved C19 16.1 mm to (114.3, 101.0)
- moved R11 16.1 mm to (118.9, 103.1)
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Routing:
- net TIA_4.5V: track 129.3 -> 4.95 mm
- net +5V: track 100.0 -> 25.7 mm
- net /ADC_CH7: track 72.0 -> 0.00 mm, vias 1 -> 0
- net /ADC_CH0: track 59.2 -> 8.44 mm
- net /ADC_CH3: track 47.4 -> 0.00 mm
- net /ADC_CH4: track 46.7 -> 0.00 mm
- net /CH6: track 53.8 -> 7.88 mm, vias 1 -> 0
- net /CH5: track 53.1 -> 7.88 mm, vias 1 -> 0
- net /CH1: track 49.1 -> 5.83 mm
- net /CH2: track 49.1 -> 5.83 mm
- net /ADC_CH6: track 40.3 -> 0.00 mm, vias 1 -> 0
- net /ADC_CH1: track 32.5 -> 0.00 mm
- net /ADC_CH2: track 26.7 -> 0.00 mm
- net /ADC_CH5: track 25.1 -> 0.00 mm
- net ADC_INT: track 23.3 -> 0.00 mm
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Other:
- board size 90 x 75 mm -> 135 x 75 mm

Commit message: update
Parts:
- moved J6 76.2 mm to (165.5, 53.6)
- moved U7 25.8 mm to (112.5, 98.1)
- moved J3 25.4 mm to (102.3, 96.0)
- moved C35 25.3 mm to (116.5, 105.1)
- moved C25 25.2 mm to (109.5, 104.1)
- moved C19 18.3 mm to (117.3, 119.1)
- moved C34 16.9 mm to (112.0, 122.9), turned to 180 degrees
- moved C11 16.0 mm to (122.3, 119.1)
- moved R11 16.0 mm to (119.8, 119.1)
- moved C29 15.9 mm to (121.3, 124.1)
- moved R19 15.2 mm to (118.8, 116.1), turned to 0 degrees
- moved C12 14.7 mm to (132.5, 120.1)
- moved C20 14.7 mm to (139.4, 120.0)
- moved R12 14.7 mm to (134.8, 120.0)
- moved R20 14.7 mm to (137.1, 120.0)
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Routing:
- net GND: track 61.8 -> 14.1 mm, vias 26 -> 12
- net /ADC_CH7: track 0.00 -> 34.6 mm, vias 0 -> 1
- net /ADC_CH3: track 0.00 -> 31.3 mm, vias 0 -> 1
- net /ADC_CH4: track 0.00 -> 30.7 mm, vias 0 -> 1
- net +5V: track 25.7 -> 0.00 mm
- net /ADC_CH0: track 8.44 -> 34.0 mm, vias 0 -> 1
- net TIA0_V: track 25.2 -> 0.00 mm
- net TIA1_V: track 23.3 -> 4.32 mm
- net PWR_MAX15V: track 14.4 -> 0.00 mm
- net ADC_SDI: track 13.9 -> 0.00 mm
- net /ADC_CH6: track 0.00 -> 8.30 mm
- net /ADC_CH1: track 0.00 -> 7.90 mm
- net /ADC_CH5: track 0.00 -> 7.53 mm
- net /ADC_CH2: track 0.00 -> 7.32 mm
- net /CH4: track 12.2 -> 5.20 mm, vias 1 -> 0
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- added copper zone on F.Cu, net +5V
- added copper zone on F.Cu, net TIA_4.5V
